File: KiCad/ACE5SMD/ACE5SMD.sch (KiCad schematic (older format))
At the start: 100 parts, among them IC1 LM7805_TO220, Q1 MMBT3904, Q3 BC847, X1 CRYSTALHC49U-V 6.556MHz, X2 5MHz

Commit message: Remove Speakrer leave 2 pin connector add single transistor amp to composite out.
Signed-off-by: John Bradley <flypie@rocketmail.com>
Parts:
- removed COMPOSITE1: Conn_01x02, Connector_PinHeader_2.54mm:PinHeader_1x02_P2.54mm_Vertical, symbol Connector_Generic:Conn_01x02
- removed SP1: Speaker, Buzzer_Beeper:PUIAudio_SMT_0825_S_4_R, symbol Device:Speaker
- added COMPOSITE-OUT1: COMPOSITE-OUT1, Connector_PinHeader_2.54mm:PinHeader_1x02_P2.54mm_Vertical, symbol Connector_Generic:Conn_01x02
- added Q4: 2N3904, Package_TO_SOT_SMD:SOT-23, symbol Transistor_BJT:2N3904
- added R110: 200, Resistor_SMD:R_0603_1608Metric, symbol Device:R
- added R111: 100, Resistor_SMD:R_0603_1608Metric, symbol Device:R
- added R112: 18, Resistor_SMD:R_0603_1608Metric, symbol Device:R
- added SPK1: SPK1, Connector_PinHeader_2.54mm:PinHeader_1x02_P2.54mm_Vertical, symbol Connector_Generic:Conn_01x02
- R32: footprint Resistor_THT:R_Axial_DIN0204_L3.6mm_D1.6mm_P2.54mm_Vertical -> Resistor_SMD:R_0603_1608Metric
- Z0: symbol z84c15qfp100:Z84C15QFP100 -> Zilog_z80:Z84C15-QFP
Connections:
- net labels added: +9Vsm
- wire segments 879 -> 885
Other:
- moved on the sheet: Z5-6, Z7-8
Changed lines of the file:
@@
 EESchema Schematic File Version 4
 LIBS:ACE5SMD-cache
+LIBS:CompsoiteAmp-cache
 EELAYER 29 0
 EELAYER END
@@
 	2100 7550 2425 7550
 $Comp
-L z84c15qfp100:Z84C15QFP100 Z0
+L Zilog_z80:Z84C15-QFP Z0
 U 1 1 09F6B21C
 P 1300 3350
@@
 $EndComp
 $Comp
-L z84c15qfp100:Z84C15QFP100 Z0
+L Zilog_z80:Z84C15-QFP Z0
 U 3 1 09F6B214
 P 1300 6750
@@
 	15800 3000 15800 2800
 Wire Wire Line
-	22500 3300 22400 3300
-Wire Wire Line
 	24375 5175 24375 5275
 Wire Wire Line
@@
 	21800 3250 21800 3200
 Connection ~ 21800 3200
-Wire Wire Line
-	21800 3200 22500 3200
 Text Label 7475 16000 2    50   ~ 0
 A15
@@
 +5V
 Text GLabel 4875 14750 0    50   Input ~ 0
-+9V
++9Vsm
 Text GLabel 9225 16725 1    50   Input ~ 0
-+9V
++9Vsm
 Text GLabel 10850 16725 1    50   Input ~ 0
 +5V
@@
 $EndComp
 $Comp
-L power:GND #PWR0138
-U 1 1 69F76E6E
-P 22400 3300
-F 0 "#PWR0138" H 22400 3050 50  0001 C CNN
-F 1 "GND" V 22385 3170 50  0000 R CNN
-F 2 "" H 22400 3300 50  0001 C CNN
-F 3 "" H 22400 3300 50  0001 C CNN
-	1    22400 3300
-	0    1    1    0
-$EndComp
-$Comp
 L power:VCC #PWR0139
 U 1 1 6A07A24C
@@
 MA18
 $Comp
-L Device:Speaker SP1
-U 1 1 5D362C49
-P 19050 12850
-F 0 "SP1" H 19240 12890 50  0000 L CNN
-F 1 "Speaker" H 19240 12790 50  0000 L CNN
-F 2 "Buzzer_Beeper:PUIAudio_SMT_0825_S_4_R" H 19050 12650 50  0001 C CNN
-F 3 "~" H 19040 12800 50  0001 C CNN
-	1    19050 12850
-	1    0    0    -1
-$EndComp
-$Comp
 L power:VCC #PWR0108
 U 1 1 5D829722
@@
 	1    0    0    -1
 $EndComp
-$Comp
-L Connector_Generic:Conn_01x02 COMPOSITE1
-U 1 1 5F41E7FB
-P 22700 3200
-F 0 "COMPOSITE1" H 22800 3200 50  0000 L CNN
-F 1 "Conn_01x02" H 22800 3100 50  0000 L CNN
-F 2 "Connector_PinHeader_2.54mm:PinHeader_1x02_P2.54mm_Vertical" H 22700 3200 50  0001 C CNN
-F 3 "~" H 22700 3200 50  0001 C CNN
-	1    22700 3200
-	1    0    0    -1
-$EndComp
 Wire Wire Line
 	17250 14000 17650 14000
@@
 $EndComp
 $Comp
-L z84c15qfp100:Z84C15QFP100 Z0
+L Zilog_z80:Z84C15-QFP Z0
 U 4 1 09F6B208
 P 1325 8050
@@
 $EndComp
 $Comp
-L z84c15qfp100:Z84C15QFP100 Z0
+L Zilog_z80:Z84C15-QFP Z0
 U 5 1 09F6B20C
 P 1325 9550
@@
 $EndComp
 $Comp
-L z84c15qfp100:Z84C15QFP100 Z0
+L Zilog_z80:Z84C15-QFP Z0
 U 7 1 09F6B204
 P 1325 12725
@@
 $EndComp
 $Comp
-L SamacSys_Parts:71321SA55JG8 Z7-8
-U 1 1 5D27DF0C
-P 21050 4675
-F 0 "Z7-8" H 22045 4970 50  0000 C CNN
-F 1 "71321SA55JG8" H 21330 4960 50  0000 C CNN
-F 2 "Package_LCC:PLCC-52" H 22300 4775 50  0001 L CNN
-F 3 "https://www.idt.com/document/dst/71321421-datasheet" H 22300 4675 50  0001 L CNN
-F 4 "IC SRAM 16K PARALLEL 52PLCC" H 22300 4575 50  0001 L CNN "Description"
-F 5 "3.63" H 22300 4475 50  0001 L CNN "Height"
-F 6 "IDT, Integrated Device Technology Inc" H 22300 4175 50  0001 L CNN "Manufacturer_Name"
-F 7 "71321SA55JG8" H 22300 4075 50  0001 L CNN "Manufacturer_Part_Number"
-	1    21050 4675
-	1    0    0    -1
-$EndComp
-$Comp
 L SamacSys_Parts:71321SA55JG8 Z5-6
 U 1 1 5D3B1412
-P 18450 5275
-F 0 "Z5-6" H 19100 5950 50  0000 C CNN
-F 1 "71321SA55JG8" H 19100 5850 50  0000 C CNN
-F 2 "Package_LCC:PLCC-52" H 19250 5925 50  0001 L CNN
-F 3 "https://www.idt.com/document/dst/71321421-datasheet" H 19250 5825 50  0001 L CNN
-F 4 "IC SRAM 16K PARALLEL 52PLCC" H 19250 6025 50  0001 L CNN "Description"
-F 5 "3.63" H 19650 5225 50  0001 L CNN "Height"
-F 6 "IDT, Integrated Device Technology Inc" H 19250 6125 50  0001 L CNN "Manufacturer_Name"
-F 7 "71321SA55JG8" H 19650 4825 50  0001 L CNN "Manufacturer_Part_Number"
-	1    18450 5275
+P 18450 5125
+F 0 "Z5-6" H 19100 5800 50  0000 C CNN
+F 1 "71321SA55JG8" H 19100 5700 50  0000 C CNN
+F 2 "Package_LCC:PLCC-52" H 19250 5775 50  0001 L CNN
+F 3 "https://www.idt.com/document/dst/71321421-datasheet" H 19250 5675 50  0001 L CNN
+F 4 "IC SRAM 16K PARALLEL 52PLCC" H 19250 5875 50  0001 L CNN "Description"
+F 5 "3.63" H 19650 5075 50  0001 L CNN "Height"
+F 6 "IDT, Integrated Device Technology Inc" H 19250 5975 50  0001 L CNN "Manufacturer_Name"
+F 7 "71321SA55JG8" H 19650 4675 50  0001 L CNN "Manufacturer_Part_Number"
+	1    18450 5125
 	1    0    0    -1
 $EndComp
@@
 	4025 8750 4825 8750
 $Comp
-L z84c15qfp100:Z84C15QFP100 Z0
+L Zilog_z80:Z84C15-QFP Z0
 U 2 1 09F6B210
 P 5025 8350
@@
 	2325 11150 2025 11150
 $Comp
-L z84c15qfp100:Z84C15QFP100 Z0
+L Zilog_z80:Z84C15-QFP Z0
 U 6 1 09F6B200
 P 1325 11050
@@
 	1    0    0    -1
 $EndComp
-Connection ~ 18250 13200
 Connection ~ 17950 13200
 Wire Wire Line
 	17950 13200 17950 13800
 Wire Wire Line
-	18250 13200 18850 13200
-Wire Wire Line
 	18250 13200 18250 13100
 Wire Wire Line
@@
 F 0 "R32" V 11000 7100 50  0000 C CNN
 F 1 "1K0" V 11100 7100 50  0000 C CNN
-F 2 "Resistor_THT:R_Axial_DIN0204_L3.6mm_D1.6mm_P2.54mm_Vertical" V 11180 7100 50  0001 C CNN
+F 2 "Resistor_SMD:R_0603_1608Metric" V 11180 7100 50  0001 C CNN
 F 3 "~" H 11250 7100 50  0001 C CNN
 	1    11250 7100
@@
 Text Label 11500 7100 0    50   ~ 0
 #WE
+$Comp
+L SamacSys_Parts:71321SA55JG8 Z7-8
+U 1 1 5D27DF0C
+P 21050 4525
+F 0 "Z7-8" H 22045 4820 50  0000 C CNN
+F 1 "71321SA55JG8" H 21330 4810 50  0000 C CNN
+F 2 "Package_LCC:PLCC-52" H 22300 4625 50  0001 L CNN
+F 3 "https://www.idt.com/document/dst/71321421-datasheet" H 22300 4525 50  0001 L CNN
+F 4 "IC SRAM 16K PARALLEL 52PLCC" H 22300 4425 50  0001 L CNN "Description"
+F 5 "3.63" H 22300 4325 50  0001 L CNN "Height"
+F 6 "IDT, Integrated Device Technology Inc" H 22300 4025 50  0001 L CNN "Manufacturer_Name"
+F 7 "71321SA55JG8" H 22300 3925 50  0001 L CNN "Manufacturer_Part_Number"
+	1    21050 4525
+	1    0    0    -1
+$EndComp
+Wire Wire Line
+	23425 3350 23425 3250
+Wire Wire Line
+	21800 3200 22500 3200
+$Comp
+L power:GND #SUPPLY0110
+U 1 1 5D703F5E
+P 23425 3250
+F 0 "#SUPPLY0110" H 23425 3250 50  0001 C CNN
+F 1 "GND" H 23350 3125 59  0000 L BNN
+F 2 "" H 23425 3250 50  0001 C CNN
+F 3 "" H 23425 3250 50  0001 C CNN
+	1    23425 3250
+	-1   0    0    1
+$EndComp
+$Comp
+L Connector_Generic:Conn_01x02 COMPOSITE-OUT1
+U 1 1 5D703F64
+P 23625 3450
+F 0 "COMPOSITE-OUT1" H 23725 3375 50  0000 L CNN
+F 1 "COMPOSITE-OUT1" H 23575 3200 50  0001 C CNN
+F 2 "Connector_PinHeader_2.54mm:PinHeader_1x02_P2.54mm_Vertical" H 23625 3450 50  0001 C CNN
+F 3 "~" H 23625 3450 50  0001 C CNN
+	1    23625 3450
+	1    0    0    1
+$EndComp
+$Comp
+L Transistor_BJT:2N3904 Q4
+U 1 1 5D703F6A
+P 22700 3200
+F 0 "Q4" H 22500 3200 59  0000 L BNN
+F 1 "2N3904" H 22300 3100 59  0000 L BNN
+F 2 "Package_TO_SOT_SMD:SOT-23" H 22700 3200 50  0001 C CNN
+F 3 "" H 22700 3200 50  0001 C CNN
+	1    22700 3200
+	1    0    0    -1
+$EndComp
+Wire Wire Line
+	22500 3450 22400 3450
+$Comp
+L power:GND #SUPPLY0111
+U 1 1 5D703F71
+P 22400 3450
+F 0 "#SUPPLY0111" H 22400 3450 50  0001 C CNN
+F 1 "GND" H 22325 3325 59  0000 L BNN
+F 2 "" H 22400 3450 50  0001 C CNN
+F 3 "" H 22400 3450 50  0001 C CNN
+	1    22400 3450
+	0    1    1    0
+$EndComp
+$Comp
+L power:VCC #P+0102
+U 1 1 5D703F77
+P 22800 2950
+F 0 "#P+0102" H 22800 2950 50  0001 C CNN
+F 1 "VCC" H 22850 3175 59  0000 C CNN
+F 2 "" H 22800 2950 50  0001 C CNN
+F 3 "" H 22800 2950 50  0001 C CNN
+	1    22800 2950
+	1    0    0    -1
+$EndComp
+Wire Wire Line
+	22800 3400 22800 3450
+Wire Wire Line
+	22800 3450 23050 3450
+Connection ~ 22800 3450
+$Comp
+L Device:R R111
+U 1 1 5D703F80
+P 22650 3450
+F 0 "R111" V 22750 3450 50  0000 C CNN
+F 1 "100" V 22850 3450 50  0000 C CNN
+F 2 "Resistor_SMD:R_0603_1608Metric" V 22580 3450 50  0001 C CNN
+F 3 "~" H 22650 3450 50  0001 C CNN
+	1    22650 3450
+	0    1    1    0
+$EndComp
+Wire Wire Line
+	22800 3000 22800 2950
+$Comp
+L Device:R R112
+U 1 1 5D703F87
+P 23200 3450
+F 0 "R112" V 22950 3450 50  0000 C CNN
+F 1 "18" V 23050 3450 50  0000 C CNN
+F 2 "Resistor_SMD:R_0603_1608Metric" V 23130 3450 50  0001 C CNN
+F 3 "~" H 23200 3450 50  0001 C CNN
+	1    23200 3450
+	0    1    1    0
+$EndComp
+Wire Wire Line
+	23425 3450 23350 3450
+$Comp
+L Connector_Generic:Conn_01x02 SPK1
+U 1 1 5E96BAA0
+P 19050 12950
+F 0 "SPK1" H 19150 12875 50  0000 L CNN
+F 1 "SPK1" H 19000 12700 50  0001 C CNN
+F 2 "Connector_PinHeader_2.54mm:PinHeader_1x02_P2.54mm_Vertical" H 19050 12950 50  0001 C CNN
+F 3 "~" H 19050 12950 50  0001 C CNN
+	1    19050 12950
+	1    0    0    1
+$EndComp
+$Comp
+L Device:R R110
+U 1 1 5E96BAA6
+P 18550 13200
+F 0 "R110" V 18300 13200 50  0000 C CNN
+F 1 "200" V 18400 13200 50  0000 C CNN
+F 2 "Resistor_SMD:R_0603_1608Metric" V 18480 13200 50  0001 C CNN
+F 3 "~" H 18550 13200 50  0001 C CNN
+	1    18550 13200
+	0    1    1    0
+$EndComp
+Wire Wire Line
+	18850 13200 18700 13200
+Wire Wire Line
+	18400 13200 18250 13200
+Connection ~ 18250 13200
 $EndSCHEMATC
