File: KiCad/ACE1/ACE1.sch (KiCad schematic (older format))
At the start: 147 parts, among them IC1 78T, Q1 2N3904, Q2 2N2369, Q3 BC183, Q4 2N3904, X1 6.556MHz

Commit message: Renumber components to match original Schema.
Parts:
- C1: renamed from C5; value 47N -> 30p
- C2: renamed from C1; value 47N -> 100
- C5: renamed from C2; value 47N -> 47p
- R1: renamed from R9; value 47k -> 4k7
- R9: renamed from R2; value 12k -> 22k
- renumbered R1 to R2
Connections:
- net VCC: now also D2.1 (K); no longer D2.2 (A)
- net at C5.1, Q3.1 (C), R100.2: now also D2.2 (A); no longer D2.1 (K)
Other:
- moved on the sheet: C1, C10, C11, C12, C13, C14, C15, C16, C17, C18, C19, C2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

Commit message: Double check transistors
Parts:
- renumbered Z18 to Z17, Z17 to Z18, Z12 to Z28, Z13 to Z29
Connections:
- net ~CLK: no longer E1.CLK (~CLK)
- net PHI: now reaches Q2.3 (C), R8.2, Z0.6 (CLK)
- net PHI: now also E1.CLK (~CLK)
Changed lines of the file:
@@
 	26025 10625 26125 10625
 Text Label 26125 10625 0    50   ~ 0
-~CLK
+PHI
 $Comp
 L 74xx:74LS00 Z19
@@
 $EndComp
 $Comp
-L 74xx:74LS138 Z13
+L 74xx:74LS138 Z29
 U 1 1 39104969
 P 6350 6875
-F 0 "Z13" H 5950 7300 59  0000 L BNN
+F 0 "Z29" H 6350 7600 59  0000 C CNN
 F 1 "74138N" H 5950 6275 59  0001 L BNN
 F 2 "Package_DIP:DIP-16_W7.62mm" H 6350 6875 50  0001 C CNN
@@
 $EndComp
 $Comp
-L 74xx:74LS367 Z17
+L 74xx:74LS367 Z18
 U 1 1 527FC48B
 P 19150 6275
-F 0 "Z17" H 18850 6800 59  0000 L BNN
+F 0 "Z18" H 18850 6800 59  0000 L BNN
 F 1 "74367N" H 18850 5575 59  0001 L BNN
 F 2 "Package_DIP:DIP-16_W7.62mm" H 19150 6275 50  0001 C CNN
@@
 $EndComp
 $Comp
-L 74xx:74LS367 Z18
+L 74xx:74LS367 Z17
 U 1 1 9B296254
 P 20850 6275
-F 0 "Z18" H 20550 6800 59  0000 L BNN
+F 0 "Z17" H 20550 6800 59  0000 L BNN
 F 1 "74367N" H 20550 5575 59  0001 L BNN
 F 2 "Package_DIP:DIP-16_W7.62mm" H 20850 6275 50  0001 C CNN
@@
 ~NMI
 $Comp
-L 74xx:74LS166 Z12
+L 74xx:74LS166 Z28
 U 1 1 D992BD4C
 P 23750 6275
-F 0 "Z12" V 24350 6275 59  0000 C CNN
+F 0 "Z28" V 24375 6275 59  0000 C CNN
 F 1 "74166N" H 23450 5375 59  0001 L BNN
 F 2 "Package_DIP:DIP-16_W7.62mm" H 23750 6275 50  0001 C CNN
@@
 	1    0    0    -1
 $EndComp
+Text Label 5975 11475 0    50   ~ 0
+PHI
 $EndSCHEMATC

Commit message: ACE2NOKBV2MK2 update IC placement. Reverse Diode.
Signed-off-by: John Bradley <flypie@rocketmail.com>
Parts:
- added KEYBOARD1: Conn_02x08_Odd_Even, Connector_PinHeader_2.54mm:PinHeader_2x08_P2.54mm_Vertical, symbol Connector_Generic:Conn_02x08_Odd_Even
Connections:
- net ROW11: now reaches D7.1 (K), S1.1, S2.1, S3.1, S4.1, S5.1
- net ROW11: now also KEYBOARD1.8 (Pin_8)
- net ROW10: now reaches D8.1 (K), S11.1, S12.1, S13.1, S14.1, S15.1
- net ROW10: now also KEYBOARD1.6 (Pin_6)
- net COLC: now reaches S13.2, S18.2, S23.2, S28.2, S3.2, S33.2, S38.2, S8.2, Z14.6 (I3)
- net COLC: now also KEYBOARD1.5 (Pin_5)
- net ROW13: now reaches D5.1 (K), S16.1, S17.1, S18.1, S19.1, S20.1
- net ROW13: now also KEYBOARD1.12 (Pin_12)
- net COLA: now reaches S1.2, S10.2, S11.2, S20.2, S21.2, S30.2, S31.2, S40.2, Z14.2 (I1)
- net COLA: now also KEYBOARD1.1 (Pin_1)
- net ROW9: now reaches D9.1 (K), S21.1, S22.1, S23.1, S24.1, S25.1
- net ROW9: now also KEYBOARD1.4 (Pin_4)
- net COLD: now reaches S14.2, S17.2, S24.2, S27.2, S34.2, S37.2, S4.2, S7.2, Z14.10 (I4)
- net COLD: now also KEYBOARD1.7 (Pin_7)
- net COLE: now reaches S15.2, S16.2, S25.2, S26.2, S35.2, S36.2, S5.2, S6.2, Z14.14 (I6)
- net COLE: now also KEYBOARD1.9 (Pin_9)
- net COLB: now reaches S12.2, S19.2, S2.2, S22.2, S29.2, S32.2, S39.2, S9.2, Z14.4 (I2)
- net COLB: now also KEYBOARD1.3 (Pin_3)
- net ROW14: now reaches D4.1 (K), S26.1, S27.1, S28.1, S29.1, S30.1
- net ROW14: now also KEYBOARD1.14 (Pin_14)
- net ROW15: now reaches D3.1 (K), S36.1, S37.1, S38.1, S39.1, S40.1
- net ROW15: now also KEYBOARD1.16 (Pin_16)
- net ROW12: now reaches D6.1 (K), S10.1, S6.1, S7.1, S8.1, S9.1
- net ROW12: now also KEYBOARD1.10 (Pin_10)
- net ROW8: now reaches D10.1 (K), S31.1, S32.1, S33.1, S34.1, S35.1
- net ROW8: now also KEYBOARD1.2 (Pin_2)
- no-connect marks 20 -> 23
Other:
- moved on the sheet: Z10C, Z11C, Z19E, Z1B, Z20E, Z21D, Z22D, Z23E, Z24E, Z25E, Z26E, Z27C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
