File: KiCad/ACE3NOKB/KIO.sch (KiCad schematic (older format))
At the start: 7 parts, among them J100 Conn_02x05_Odd_Even, J101 Conn_02x05_Odd_Even, J102 Conn_02x05_Odd_Even, J103 Conn_02x03_Odd_Even, J104 Conn_02x03_Odd_Even, J105 Conn_02x04_Odd_Even

Commit message: Latest changes fix Diode misake in 2NOKB.
Signed-off-by: John Bradley <flypie@rocketmail.com>
Parts:
- J100, J101, J102: Manufacturer_Part_Number TSW–105–10–T–D–RA -> HTSW-105-08-S-D
- J103, J104: Manufacturer_Part_Number TSW–103–10–T–D–RA -> TSW-103-08-S-D
- J105: Manufacturer_Name SAMTEC -> TE Connectivity / AMP; Manufacturer_Part_Number TSW–104–10–T–D–RA -> 5-146250-2
Changed lines of the file:
@@
 F 2 "Connector_PinHeader_2.54mm:PinHeader_2x04_P2.54mm_Vertical" H 2550 5525 50  0001 C CNN
 F 3 "" H 2550 5525 50  0001 C CNN
-F 4 "SAMTEC" H 2550 5525 50  0001 C CNN "Manufacturer_Name"
-F 5 "TSW–104–10–T–D–RA" H 2550 5525 50  0001 C CNN "Manufacturer_Part_Number"
+F 4 "TE Connectivity / AMP" H 2550 5525 50  0001 C CNN "Manufacturer_Name"
+F 5 "5-146250-2" H 2550 5525 50  0001 C CNN "Manufacturer_Part_Number"
 	1    2550 5525
 	1    0    0    -1
@@
 F 3 "" H 2550 4925 50  0001 C CNN
 F 4 "SAMTEC" H 2550 4925 50  0001 C CNN "Manufacturer_Name"
-F 5 "TSW–103–10–T–D–RA" H 2550 4925 50  0001 C CNN "Manufacturer_Part_Number"
+F 5 "TSW-103-08-S-D" H 2550 4925 50  0001 C CNN "Manufacturer_Part_Number"
 	1    2550 4925
 	1    0    0    -1
@@
 F 3 "" H 2550 4325 50  0001 C CNN
 F 4 "SAMTEC" H 2550 4325 50  0001 C CNN "Manufacturer_Name"
-F 5 "TSW–103–10–T–D–RA" H 2550 4325 50  0001 C CNN "Manufacturer_Part_Number"
+F 5 "TSW-103-08-S-D" H 2550 4325 50  0001 C CNN "Manufacturer_Part_Number"
 	1    2550 4325
 	1    0    0    -1
@@
 F 3 "" H 2525 1925 50  0001 C CNN
 F 4 "SAMTEC" H 2525 1925 50  0001 C CNN "Manufacturer_Name"
-F 5 "TSW–105–10–T–D–RA" H 2525 1925 50  0001 C CNN "Manufacturer_Part_Number"
+F 5 "HTSW-105-08-S-D" H 2525 1925 50  0001 C CNN "Manufacturer_Part_Number"
 	1    2525 1925
 	1    0    0    -1
@@
 F 3 "" H 2525 2725 50  0001 C CNN
 F 4 "SAMTEC" H 2525 2725 50  0001 C CNN "Manufacturer_Name"
-F 5 "TSW–105–10–T–D–RA" H 2525 2725 50  0001 C CNN "Manufacturer_Part_Number"
+F 5 "HTSW-105-08-S-D" H 2525 2725 50  0001 C CNN "Manufacturer_Part_Number"
 	1    2525 2725
 	1    0    0    -1
@@
 F 3 "" H 2525 3525 50  0001 C CNN
 F 4 "SAMTEC" H 2525 3525 50  0001 C CNN "Manufacturer_Name"
-F 5 "TSW–105–10–T–D–RA" H 2525 3525 50  0001 C CNN "Manufacturer_Part_Number"
+F 5 "HTSW-105-08-S-D" H 2525 3525 50  0001 C CNN "Manufacturer_Part_Number"
 	1    2525 3525
 	1    0    0    -1

Commit message: This version sent off for production.
Fix from last mistakes.

3 74xx383s replaced with 2 *74xx4040. See https://github.com/ricaflops/Jupiter-II

Memory map reverted back to orginal as far as RAM is concerned. ROM space 5k added overlapping the write only portions of char RAM and none docded 3k. Total 5k.


https://www.tindie.com/products/tynemouthsw/minstrel-4th-z80-computer-kit/



Signed-off-by: John Bradley <flypie@rocketmail.com>
Parts:
- J100, J101, J102: value Conn_02x05_Odd_Even -> Conn_02x06_Odd_Even; footprint Connector_PinHeader_2.54mm:PinHeader_2x05_P2.54mm_Vertical -> Connector_PinHeader_2.54mm:PinHeader_2x06_P2.54mm_Vertical; symbol Connector_Generic:Conn_02x05_Odd_Even -> Connector_Generic:Conn_02x06_Odd_Even; Manufacturer_Part_Number HTSW-105-08-S-D -> HTSW-106-08-S-D
- J103, J104: value Conn_02x03_Odd_Even -> Conn_02x04_Odd_Even; footprint Connector_PinHeader_2.54mm:PinHeader_2x03_P2.54mm_Vertical -> Connector_PinHeader_2.54mm:PinHeader_2x04_P2.54mm_Vertical; symbol Connector_Generic:Conn_02x03_Odd_Even -> Connector_Generic:Conn_02x04_Odd_Even; Manufacturer_Part_Number TSW-103-08-S-D -> TSW-104-08-S-D
- J105: value Conn_02x04_Odd_Even -> Conn_02x05_Odd_Even; footprint Connector_PinHeader_2.54mm:PinHeader_2x04_P2.54mm_Vertical -> Connector_PinHeader_2.54mm:PinHeader_2x05_P2.54mm_Vertical; symbol Connector_Generic:Conn_02x04_Odd_Even -> Connector_Generic:Conn_02x05_Odd_Even; Manufacturer_Part_Number 5-146250-2 -> HTSW-105-08-S-D
Connections:
- net GND: now also J100.12 (Pin_12), J101.12 (Pin_12), J102.12 (Pin_12), J103.8 (Pin_8), J104.8 (Pin_8), J105.10 (Pin_10)
- net VCC: now also J100.11 (Pin_11), J101.11 (Pin_11), J102.11 (Pin_11), J103.7 (Pin_7), J104.7 (Pin_7), J105.9 (Pin_9)
