File: KiCad/ACE3NOKB/ACE3NOKB.sch (KiCad schematic (older format))
At the start: 97 parts, among them J5 Conn_01x12_Female, J6 Conn_01x09_Female, J7 Conn_01x03, J8 Conn_02x05, Q1 2N3904, Q101 2N3904, Q2 2N2369, X1 6.5MHz

Commit message: This version sent off for production.
Fix from last mistakes.

3 74xx383s replaced with 2 *74xx4040. See https://github.com/ricaflops/Jupiter-II

Memory map reverted back to orginal as far as RAM is concerned. ROM space 5k added overlapping the write only portions of char RAM and none docded 3k. Total 5k.


https://www.tindie.com/products/tynemouthsw/minstrel-4th-z80-computer-kit/



Signed-off-by: John Bradley <flypie@rocketmail.com>
Parts:
- POWER-9V-DC1: value cuipj:CUI_PJ-036C -> 163-179PH-EX; footprint cuipj:CUI_PJ-036C -> SamacSys_Parts:163179PHEX; symbol Connector:Barrel_Jack -> SamacSys_Parts:163-179PH-EX
Connections:
- net GND: now also POWER-9V-DC1.C; no longer POWER-9V-DC1.2
- net VIDEO: now also D1.2 (A), Q101.2 (B), R3.1, R4.1
- net at C10.2, C9.1, L1.1: now also POWER-9V-DC1.B; no longer POWER-9V-DC1.1
- net SYNCLEVEL: now reaches D1.1 (K), Z25.4
- net HSYNC: now reaches Z22.12, Z25.5
Other:
- moved on the sheet: C1, C2, C4, C7, Q1, Q2, R1, R110, R130, R131, R2, R24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

Commit message: Rotate a single transistor as was EBC not CBE.
Signed-off-by: John Bradley <flypie@rocketmail.com>
Connections:
- net 50Hz renamed CLK\TRG3
- no-connect marks 19 -> 20
Changed lines of the file:
@@
 $EndComp
 $Comp
-L power:PWR_FLAG #~FLG0102
-U 1 1 727010D5
-P 1950 14650
-F 0 "#~FLG0102" H 1950 14725 50  0001 C CNN
-F 1 "PWR_FLAG" V 1950 14825 50  0000 L CNN
-F 2 "" H 1950 14650 50  0001 C CNN
-F 3 "" H 1950 14650 50  0001 C CNN
-	1    1950 14650
-	1    0    0    -1
-$EndComp
-$Comp
 L power:GND #~PWR0152
 U 1 1 6AC5A37D
@@
 Wire Wire Line
 	19675 10350 20025 10350
-Text GLabel 20025 10350 3    50   Input ~ 0
-50Hz
 Text GLabel 18400 13750 0    50   Input ~ 0
 BASECLK_DIV_32
@@
 NoConn ~ 9825 8450
 Wire Wire Line
-	1550 14650 1950 14650
-Wire Wire Line
 	1625 15400 1625 15450
 Wire Wire Line
 	1625 15450 1550 15450
-$Comp
-L power:PWR_FLAG #~FLG0101
-U 1 1 725FB0E7
-P 1975 15400
-F 0 "#~FLG0101" H 1975 15475 50  0001 C CNN
-F 1 "PWR_FLAG" V 1975 15575 50  0000 L CNN
-F 2 "" H 1975 15400 50  0001 C CNN
-F 3 "" H 1975 15400 50  0001 C CNN
-	1    1975 15400
-	-1   0    0    1
-$EndComp
-Connection ~ 1975 15400
-Wire Wire Line
-	1975 15400 1625 15400
-Connection ~ 1950 14650
-Wire Wire Line
-	1975 15400 2475 15400
-Wire Wire Line
-	1950 14650 2825 14650
 Text Label 20125 9500 1    50   ~ 0
 HSYNC
@@
 Text Label 20300 13350 0    50   ~ 0
 CNT0
+Wire Wire Line
+	1625 15400 2475 15400
+Wire Wire Line
+	1550 14650 2825 14650
+NoConn ~ 1450 15450
+Text Label 20025 10350 3    50   ~ 0
+50Hz
 $EndSCHEMATC
