File: KiCad/ACE3NOKB/Cascade393.sch (KiCad schematic (older format))
At the start: 9 parts

Commit message: Update ACE3NOKB to reflect errors in Mem Decode. ACE5NOKB test SMT ideas. Added 180 & 380.
Signed-off-by: John Bradley <flypie@rocketmail.com>
Parts:
- renumbered Z9 to Z?, Z10 to Z?, Z11 to Z?
Changed lines of the file:
@@
 U 3 1 6C8C25AB
 P 6925 3025
-AR Path="/6C8C25AB" Ref="Z?"  Part="3"
-AR Path="/5EE121BD/6C8C25AB" Ref="Z9"  Part="3"
 F 0 "Z9" H 7155 3115 50  0000 L CNN
 F 1 "CD74HCT393E " H 7155 3015 50  0000 L CNN
@@
 U 3 1 6C8C25B3
 P 7900 3025
-AR Path="/6C8C25B3" Ref="Z?"  Part="3"
-AR Path="/5EE121BD/6C8C25B3" Ref="Z10"  Part="3"
 F 0 "Z10" H 8130 3115 50  0000 L CNN
 F 1 "CD74HCT393E " H 8130 3015 50  0000 L CNN
@@
 U 3 1 6C8C25BB
 P 8915 3025
-AR Path="/6C8C25BB" Ref="Z?"  Part="3"
-AR Path="/5EE121BD/6C8C25BB" Ref="Z11"  Part="3"
 F 0 "Z11" H 9145 3115 50  0000 L CNN
 F 1 "CD74HCT393E " H 9145 3015 50  0000 L CNN
