File: KiCad/ACE3NOKB/ACE3NOKB.kicad_sch (KiCad schematic)
At the start: 42 parts, among them J306 Conn_01x03, J307 Conn_02x05, J308 Conn_01x12_Female, J309 Conn_01x09_Female, Q1 2N3904, Q2 2N2369, X1 6.5536 MHz

Commit message: First complete system. Unlikely to work but will serve as the basis of a system to test VGA.
Signed-off-by: John Bradley <flypie@rocketmail.com>
Parts:
- added Z19: SN74AHCT00N, Package_DIP:DIP-14_W7.62mm, symbol 74xx:74LS00
- added unit 1 of Z306
- RST1: footprint TS026660BK100SCRD -> ExtraFootprints:TE Connectivity 1-1825910-4 Black Button Tactile Switch, Single Pole Single Throw (SPST)
Connections:
- net EOL renamed SCREENX5
- no-connect marks 22 -> 27
Other:
- moved on the sheet: J308, J309, Z3-4

Commit message: Update to latest symbols. Change name of Data Bus from DA to D.
Signed-off-by: John Bradley <flypie@rocketmail.com>
Parts:
- Z80CPUOUT1: symbol Connector_Generic:Conn_02x22_Odd_Even -> edg-con-ja:EDG-CON-JA-PIN
Connections:
- net +5V is gone; now on net VCC: Z80CPUOUT1.37 (+5V)
- net DA0 renamed D0
- net DA1 renamed D1
- net DA2 renamed D2
- net DA3 renamed D3
- net DA4 renamed D4
- net DA5 renamed D5
- net DA6 renamed D6
- net DA7 renamed D7
Other:
- moved on the sheet: C1, C2, C22, C4, D12, H1, H2, H3, H4, J306, J307, J308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

Commit message: Consolidation with increased configuration of speed and Int Routing to allow Orginal ACE ROM.
Signed-off-by: John Bradley <flypie@rocketmail.com>
Parts:
- removed J306: Conn_01x03, Connector_PinHeader_2.54mm:PinHeader_1x03_P2.54mm_Vertical, symbol Connector_Generic:Conn_01x03
- removed Z19: SN74AHCT00N, Package_DIP:DIP-14_W7.62mm, symbol 74xx:74LS00
- removed unit 1 of Z306
- added C8: 2200pF, Capacitor_THT:C_Disc_D5.0mm_W2.5mm_P2.50mm, symbol Device:C
- added J306: Conn_02x05_Odd_Even, Connector_PinHeader_2.54mm:PinHeader_2x05_P2.54mm_Vertical, symbol Connector_Generic:Conn_02x05_Odd_Even
- added J310, J312: Conn_01x03, Connector_PinHeader_2.54mm:PinHeader_1x03_P2.54mm_Vertical, symbol Connector_Generic:Conn_01x03
- added J311: Conn_02x01_Odd_Even, Connector_PinHeader_2.54mm:PinHeader_2x01_P2.54mm_Vertical, symbol Connector_Generic:Conn_01x02
- added R131, R303: 10K, Resistor_THT:R_Axial_DIN0204_L3.6mm_D1.6mm_P1.90mm_Vertical, symbol Device:R
- added R301, R304: 1K0, Resistor_THT:R_Axial_DIN0204_L3.6mm_D1.6mm_P1.90mm_Vertical, symbol Device:R
- added unit 3 of Z310
- C1: Manufacturer_Name AVX -> (none); Manufacturer_Part_Number SR151A300JAR -> (none)
- C2: Manufacturer_Name TDK -> (none); Manufacturer_Part_Number FA18C0G1H101JNU06 -> (none)
- C4: Manufacturer_Name tdk -> (none); Manufacturer_Part_Number FA18C0G1H470JNU00 -> (none)
- E1: renamed from Z80CPUOUT1; Manufacturer_Name HARWIN -> (none); Manufacturer_Part_Number M20-9721146 -> (none)
- H1, H2, H3, H4: Manufacturer_Name hole -> (none); Manufacturer_Part_Number hole -> (none)
- J307: value Conn_02x05 -> Conn_02x05_Odd_Even; Manufacturer_Name HARWIN -> (none); Manufacturer_Part_Number M52-040023V0545 -> (none)
- J308: footprint Connector_PinSocket_2.54mm:PinSocket_1x12_P2.54mm_Vertical -> Connector_PinHeader_2.54mm:PinHeader_1x12_P2.54mm_Vertical; symbol Connector:Conn_01x12_Female -> Connector_Generic:Conn_01x12; Manufacturer_Name HARWIN -> (none); Manufacturer_Part_Number M52-5000845 -> (none)
- J309: footprint Connector_PinSocket_2.54mm:PinSocket_1x09_P2.54mm_Vertical -> Connector_PinHeader_2.54mm:PinHeader_1x09_P2.54mm_Vertical; symbol Connector:Conn_01x09_Female -> Connector_Generic:Conn_01x09; Manufacturer_Name HARWIN -> (none); Manufacturer_Part_Number M52-5000545 -> (none)
- Logo1, Logo2: Manufacturer_Name logo -> (none); Manufacturer_Part_Number logo -> (none)
- Q1: Manufacturer_Part_Number 2N3904 -> (none)
- Q2: Manufacturer_Part_Number 2N2369 -> (none)
- R1: value 4k7 -> 4K7; Manufacturer_Name Vishay -> (none); Manufacturer_Part_Number MBA02040C4708FRP00 -> (none)
- R110, R130, R141, R24: value 10k -> 10K; Manufacturer_Name Vishay -> (none); Manufacturer_Part_Number MBA02040C1002FRP00 -> (none)
- R12: value 1k -> 1K0
- R2: value 47k -> 47K; Manufacturer_Name Vishay -> (none); Manufacturer_Part_Number MBA02040C4702FC100 -> (none)
- R7: value 1K -> 1K0; Manufacturer_Name Vishay -> (none); Manufacturer_Part_Number MBA02040C1202FRP00 -> (none)
- R8: value 270R -> 270; Manufacturer_Name Vishay -> (none); Manufacturer_Part_Number MBA02040C2700FRP00 -> (none)
- RST1: Manufacturer_Name CUI Inc. -> (none); Manufacturer_Part_Number TS02-66-60-BK-100-SCR-D -> (none); Mouser Price/Stock https://www.mouser.co.uk/ProductDetail/CUI-Devices/TS02-66-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 -> (none)
- X1: Manufacturer_Name ECS -> (none); Manufacturer_Part_Number ECS-65-20-4X -> (none)
- Z0: Manufacturer_Name Zilog -> (none); Manufacturer_Part_Number Z84C00 -> (none)
- Z1-2: Manufacturer_Name microchip -> (none); Manufacturer_Part_Number SST39SF010A-45-4I-NHE -> (none)
- Z23: Manufacturer_Name Texas Instruments -> (none); Manufacturer_Part_Number SN74AHCT86N -> (none)
- Z25: value SN74AHCT02N -> SN74AHCT02; Manufacturer_Name Texas Instruments -> (none); Manufacturer_Part_Number SN74AHCT02N -> (none)
- Z3-4, Z309: Arrow Part Number IS62C256AL-45ULI -> (none); Arrow Price/Stock https://www.arrow.com/en/products/is62c256al-45uli/integrat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 -> (none); Manufacturer_Name Integrated Silicon Solution Inc. -> (none); Manufacturer_Part_Number IS62C256AL-45ULI -> (none); Mouser Price/Stock https://www.mouser.co.uk/ProductDetail/ISSI/IS62C256AL-45UL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 -> (none)
- Z301: Manufacturer_Name Texas Instruments -> (none); Manufacturer_Part_Number SN74AS21N -> (none)
- Z302: value SN74AHCT02 -> SN74AHCT02N; Manufacturer_Name Texas Instruments -> (none); Manufacturer_Part_Number SN74AHCT32N -> (none)
- Z306: Manufacturer_Name Texas Instruments -> (none); Manufacturer_Part_Number SN74AHCT04N -> (none)
- Z307: Manufacturer_Name Texas Instruments -> (none); Manufacturer_Part_Number SN74AHCT139N -> (none)
- Z308: Manufacturer_Name Texas Instruments -> (none); Manufacturer_Part_Number SN74ALS30AN -> (none)
- Z310: value 74LS32 -> SN74AHCT32N
Connections:
- net A14: no longer Z3-4.1 (A14)
- net BASECLK: now also J306.1 (Pin_1)
- net BASECLK_DIV_16: now also J306.9 (Pin_9)
- net BASECLK_DIV_2: now also J306.3 (Pin_3)
- net BASECLK_DIV_4: now also J306.5 (Pin_5)
- net BASECLK_DIV_8: now also J306.7 (Pin_7)
- net CPUCLK: now also J306.10 (Pin_10), J306.2 (Pin_2), J306.4 (Pin_4), J306.6 (Pin_6), J306.8 (Pin_8)
- net GND: now also C8.1, J311.2 (Pin_2), R301.1, R304.2; no longer Z1-2.2 (A16)
- net VCC: now also R131.1, R303.1
- net ~{INT}: now also J310.2 (Pin_2)
- net ~{WAIT}: now also C8.2, R131.2
- net at R302.2, RST1.3 (COM_1), RST1.4 (COM_2): now also J311.1 (Pin_1)
- new net: R304.1, Z1-2.2 (A16)
- new net: J312.1 (Pin_1), R301.2
- new net: J312.3 (Pin_3), R303.2
- new net UPPERROMSELECT: J312.2 (Pin_2), Z3-4.1 (A14)
- new net V_SYNC_PULSE(50Hz): J310.3 (Pin_3)
- new net ~{INTFROMKIO}: J310.1 (Pin_1)
- no-connect marks 27 -> 25
Other:
- note added: "Mode 2 via KIO"
- note added: "Orginal int. Straight to CPU."
- moved on the sheet: C1, C2, C22, D12, H1, H2, H3, H4, J307, Logo1, Logo2, Q1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

Commit message: Fix mistake with ROM Select.
Signed-off-by: John Bradley <flypie@rocketmail.com>
Parts:
- removed R304: 1K0, Resistor_THT:R_Axial_DIN0204_L3.6mm_D1.6mm_P1.90mm_Vertical, symbol Device:R
- removed unit 4 of Z306
- removed Z307: SN74AHCT139N, Package_DIP:DIP-16_W7.62mm, symbol 74xx:74LS139
- removed Z308: SN74ALS30AN, Package_DIP:DIP-14_W7.62mm, symbol 74xx-FIX:74LS30
- added J313, J314: Conn_01x03, Connector_PinHeader_2.54mm:PinHeader_1x03_P2.54mm_Vertical, symbol Connector_Generic:Conn_01x03
- R301: value 1K0 -> 500
- R303: value 10K -> 15K
Connections:
- net A14: now also Z3-4.1 (A14); no longer Z1-2.29 (A14)
- net A15: no longer Z1-2.3 (A15)
- net UPPERROMSELECT2: now reaches Z1-2.2 (A16)
- net UPPERROMSELECT2: now also J314.2 (Pin_2)
- net at J312.1 (Pin_1), R301.2: now also J313.1 (Pin_1), J314.1 (Pin_1)
- net at J312.3 (Pin_3), R303.2: now also J313.3 (Pin_3), J314.3 (Pin_3)
- net UPPERROMSELECT renamed UPPERROMSELECT0
- net UPPERROMSELECT0: now also Z1-2.29 (A14); no longer Z3-4.1 (A14)
- new net UPPERROMSELECT1: J313.2 (Pin_2), Z1-2.3 (A15)
- no-connect marks 25 -> 23
Other:
- moved on the sheet: C1, C2, J310, J312, Q1, R1, R2, R301, R303, X1, Z25C, Z309

Commit message: Update to last expermintal version. Uses clock sythsiser and can be switched between full ACE compatible and inhanced IO. Should be able to switch between multiple ROM images tosred on the same chip.
Signed-off-by: John Bradley <flypie@rocketmail.com>
Parts:
- removed C1: 30pF, Capacitor_THT:C_Disc_D5.0mm_W2.5mm_P2.50mm, symbol Device:C_Small
- removed C2: 100pF, Capacitor_THT:C_Disc_D5.0mm_W2.5mm_P2.50mm, symbol Device:C_Small
- removed C4: 47pF, Capacitor_THT:C_Disc_D5.0mm_W2.5mm_P2.50mm, symbol Device:C
- removed J306, J307: Conn_02x05_Odd_Even, Connector_PinHeader_2.54mm:PinHeader_2x05_P2.54mm_Vertical, symbol Connector_Generic:Conn_02x05_Odd_Even
- removed J308: Conn_01x12_Female, Connector_PinHeader_2.54mm:PinHeader_1x12_P2.54mm_Vertical, symbol Connector_Generic:Conn_01x12
- removed J309: Conn_01x09_Female, Connector_PinHeader_2.54mm:PinHeader_1x09_P2.54mm_Vertical, symbol Connector_Generic:Conn_01x09
- removed Q1: 2N3904, Package_TO_SOT_THT:TO-92_Inline, symbol Transistor_BJT:2N3904
- removed Q2: 2N2369, Package_TO_SOT_THT:TO-18-3, symbol Device:Q_NPN_EBC
- removed R7: 1K0, Resistor_THT:R_Axial_DIN0204_L3.6mm_D1.6mm_P1.90mm_Vertical, symbol Device:R
- removed R8: 270, Resistor_THT:R_Axial_DIN0204_L3.6mm_D1.6mm_P1.90mm_Vertical, symbol Device:R
- removed Z23: SN74AHCT86N, Package_DIP:DIP-14_W7.62mm, symbol 74xx:74LS86
- removed Z25: SN74AHCT02, Package_DIP:DIP-14_W7.62mm, symbol 74xx:74LS02
- removed Z302: SN74AHCT02N, Package_DIP:DIP-14_W7.62mm, symbol 74xx:74LS02
- added J308, J309: Conn_01x03, Connector_PinHeader_2.54mm:PinHeader_1x03_P2.54mm_Vertical, symbol Connector_Generic:Conn_01x03
- added R306, R307: R, Resistor_THT:R_Axial_DIN0204_L3.6mm_D1.6mm_P1.90mm_Vertical, symbol Device:R
- added SW302: EG2305, ExtraFootprints:SP112DP3T, symbol ExtraSymbols:SP112-DP3T
- added Z19: SN74AHCT00N, Package_DIP:DIP-14_W7.62mm, symbol 74xx:74LS00
- added Z306: SN74AHCT04N, Package_DIP:DIP-14_W7.62mm, symbol 74xx:74LS04
- added Z312: 512MLF, Package_SO:SOIC-8_3.9x4.9mm_P1.27mm, symbol ExtraSymbols:512MLF
- R2: value 47K -> 4K7
- RST1: footprint ExtraFootprints:TE Connectivity 1-1825910-4 Black Button Tactile Switch, Single Pole Single Throw (SPST) -> ExtraFootprints:TS026660BK100SCRD; Manufacturer_Name (none) -> CUI Inc.; Manufacturer_Part_Number (none) -> TS02-66-60-BK-100-SCR-D; Mouser Price/Stock (none) -> https://www.mouser.co.uk/ProductDetail/CUI-Devices/TS02-66-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
- Z0: value Z80CPU_LCC -> Z80CPU-LCC; symbol Zilog_Z80:Z80CPU-LCC -> CPU_Zilog_Z80:Z80CPU-PLCC; Manufacturer_Name (none) -> Zilog; Manufacturer_Part_Number (none) -> Z84C00
- Z3-4, Z309: Arrow Part Number (none) -> IS62C256AL-45ULI; Arrow Price/Stock (none) -> https://www.arrow.com/en/products/is62c256al-45uli/integrat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; Manufacturer_Name (none) -> Integrated Silicon Solution Inc.; Manufacturer_Part_Number (none) -> IS62C256AL-45ULI; Mouser Price/Stock (none) -> https://www.mouser.co.uk/ProductDetail/ISSI/IS62C256AL-45UL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
Connections:
- net FONTCHARX0: now also SW302.4 (C), SW302.5 (C)
- net GND: now also R306.1, SW302.10 (M), SW302.11 (M), SW302.12 (M), SW302.9 (M), Z312.3 (GND); no longer Z0.33 (GND)
- net PHI: now also SW302.2 (COM), SW302.7 (COM)
- net SHIFTCLK: now also R1.2, X1.2, SW302.3 (B), SW302.6 (B), Z306.2, Z312.1 (X1/CLK)
- net VCC: now also R307.1, Z312.2 (VDD); no longer R1.1, Z0.13 (+5V)
- net at R2.1, X1.1: now also Z306.1
- net at R2.2: now also R1.1, Z306.2, Z306.1; no longer R1.2
- net RESET_SW: now reaches J311.1 (Pin_1), R302.2, RST1.3 (COM_1), RST1.4 (COM_2)
- new net: J308.3 (Pin_3), J309.3 (Pin_3), R307.2
- new net: J308.1 (Pin_1), J309.1 (Pin_1), R306.2
- new net S0: J308.2 (Pin_2), Z312.6 (S0)
- new net S1: J309.2 (Pin_2), Z312.7 (S1)
- new net TURBOCPUCLK: SW302.1 (A), SW302.8 (A), Z312.5 (CLKOUT)
- no-connect marks 23 -> 11
Other:
- note added: "PIN Compatible with NB3N502DR2G Different Multiply Table"
- note added: "S0 S1 CLK 0 0 4X input M 0 5.333X input 1 0 5X input 0 M 2.5X input M M 2X input 1 M 3.333X input 0 1 6X input M 1 3X input 1 1 8X input 0 = connect directly to ground 1 = connect directly to VDD M = leave unconnected (floating)"
- moved on the sheet: E1, J310, J312, J313, J314, R1, R141, R2, R301, R303, X1, Z1-2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

Commit message: Some surface mounted devices and 1G gates for space. Switch able bwteen speeds and witha Freuqency Multiplier to augment the orginal crystal.
Signed-off-by: John Bradley <flypie@rocketmail.com>
Parts:
- removed J308, J309: Conn_01x03, Connector_PinHeader_2.54mm:PinHeader_1x03_P2.54mm_Vertical, symbol Connector_Generic:Conn_01x03
- removed R1, R2: 4K7, Resistor_THT:R_Axial_DIN0204_L3.6mm_D1.6mm_P1.90mm_Vertical, symbol Device:R
- removed R306, R307: R, Resistor_THT:R_Axial_DIN0204_L3.6mm_D1.6mm_P1.90mm_Vertical, symbol Device:R
- removed SW302: EG2305, ExtraFootprints:SP112DP3T, symbol ExtraSymbols:SP112-DP3T
- removed X1: 6.5536 MHz, Crystal:Crystal_HC49-U_Vertical, symbol Device:Crystal
- removed Z306 (x2): SN74AHCT04N, Package_DIP:DIP-14_W7.62mm, symbol 74xx:74LS04
- removed Z312: 512MLF, Package_SO:SOIC-8_3.9x4.9mm_P1.27mm, symbol ExtraSymbols:512MLF
- added Z301: SN74AHCT04N, Package_DIP:DIP-14_W7.62mm, symbol 74xx:74LS04
- H301: renamed from H1; now left out of the parts list
- H302: renamed from H3; now left out of the parts list
- H303: renamed from H2; now left out of the parts list
- H304: renamed from H4; now left out of the parts list
- renumbered C22 to C301, C8 to C304, D12 to D301, E1 to E301, J311 to J301, J310 to J304, J312 to J305, J313 to J306, J314 to J307, Logo1 to Logo301, Logo2 to Logo302, R302 to R301, R12 to R302, R141 to R305, R301 to R306, R303 to R307, R130 to R308, R110 to R309, R24 to R310, R131 to R311, RST1 to RST301, Z1-2 to Z1-301, Z3-4 to Z3-301, Z310 to Z302, Z19 to Z303, Z0 to Z304, Z301 to Z305, Z309 to Z308
Connections:
- no-connect marks 11 -> 13
Other:
- added sheet CLOCK (CLOCK.kicad_sch)
- added sheet KEYBOARD (KEYBOARD.kicad_sch)
- note removed: "PIN Compatible with NB3N502DR2G Different Multiply Table"
- note removed: "S0 S1 CLK 0 0 4X input M 0 5.333X input 1 0 5X input 0 M 2.5X input M M 2X input 1 M 3.333X input 0 1 6X input M 1 3X input 1 1 8X input 0 = connect directly to ground 1 = connect directly to VDD M = leave unconnected (floating)"
- moved on the sheet: Z302C, Z302D, Z303D

Commit message: Update, with new Clock Multiplier and Wait functionality.
Signed-off-by: John Bradley <flypie@rocketmail.com>
Parts:
- removed C304: 2200pF, Capacitor_THT:C_Disc_D5.0mm_W2.5mm_P2.50mm, symbol Device:C
- removed R311: 10K, Resistor_THT:R_Axial_DIN0204_L3.6mm_D1.6mm_P1.90mm_Vertical, symbol Device:R
- removed unit 1 of Z301
- removed Z303: SN74AHCT00N, Package_DIP:DIP-14_W7.62mm, symbol 74xx:74LS00
- added C8: 47pf, Capacitor_THT:C_Disc_D3.0mm_W2.0mm_P2.50mm, symbol Device:C
- added D303, D304: 1N4148, Diode_THT:D_DO-35_SOD27_P2.54mm_Vertical_AnodeUp, symbol Diode:1N4148
- added R309: 2K, Resistor_THT:R_Axial_DIN0204_L3.6mm_D1.6mm_P2.54mm_Vertical, symbol Device:R
- added R336: 10K, Resistor_THT:R_Axial_DIN0204_L3.6mm_D1.6mm_P2.54mm_Vertical, symbol Device:R
- added R337: 1K0, Resistor_THT:R_Axial_DIN0204_L3.6mm_D1.6mm_P2.54mm_Vertical, symbol Device:R
- added R338: 330, Resistor_THT:R_Axial_DIN0204_L3.6mm_D1.6mm_P2.54mm_Vertical, symbol Device:R
- added Z19: SN74AHCT00N, Package_DIP:DIP-14_W7.62mm, symbol 74xx-FIX:74LS00
- added unit 1 of Z30
- added unit 6 of Z30
- added Z309: 74AHCT74, Package_SO:SOIC-14_3.9x8.7mm_P1.27mm, symbol 74xx-FIX:74LS74
- R12: renamed from R302; footprint Resistor_THT:R_Axial_DIN0204_L3.6mm_D1.6mm_P1.90mm_Vertical -> Resistor_THT:R_Axial_DIN0204_L3.6mm_D1.6mm_P2.54mm_Vertical
- R200: renamed from R305; footprint Resistor_THT:R_Axial_DIN0204_L3.6mm_D1.6mm_P1.90mm_Vertical -> Resistor_THT:R_Axial_DIN0204_L3.6mm_D1.6mm_P2.54mm_Vertical
- R301: footprint Resistor_THT:R_Axial_DIN0204_L3.6mm_D1.6mm_P1.90mm_Vertical -> Resistor_THT:R_Axial_DIN0204_L3.6mm_D1.6mm_P2.54mm_Vertical
- R304: renamed from R306; footprint Resistor_THT:R_Axial_DIN0204_L3.6mm_D1.6mm_P1.90mm_Vertical -> Resistor_THT:R_Axial_DIN0204_L3.6mm_D1.6mm_P2.54mm_Vertical
- R305: renamed from R307; footprint Resistor_THT:R_Axial_DIN0204_L3.6mm_D1.6mm_P1.90mm_Vertical -> Resistor_THT:R_Axial_DIN0204_L3.6mm_D1.6mm_P2.54mm_Vertical
- R306: renamed from R308; footprint Resistor_THT:R_Axial_DIN0204_L3.6mm_D1.6mm_P1.90mm_Vertical -> Resistor_THT:R_Axial_DIN0204_L3.6mm_D1.6mm_P2.54mm_Vertical
- R307: renamed from R309; footprint Resistor_THT:R_Axial_DIN0204_L3.6mm_D1.6mm_P1.90mm_Vertical -> Resistor_THT:R_Axial_DIN0204_L3.6mm_D1.6mm_P2.54mm_Vertical
- R308: renamed from R310; footprint Resistor_THT:R_Axial_DIN0204_L3.6mm_D1.6mm_P1.90mm_Vertical -> Resistor_THT:R_Axial_DIN0204_L3.6mm_D1.6mm_P2.54mm_Vertical
- Z0: renamed from Z304; value Z80CPU-LCC -> Z80CPU-PLCC
- Z1-2: renamed from Z1-301; value SST39SF010A-45-4I-NHE -> SST39SF010A-45-4I-NHE
- Z301: renamed from Z302; symbol 74xx:74LS32 -> 74xx-FIX:74LS32
- renumbered C301 to C23, D301 to D12, J304 to J302, J305 to J303, J306 to J304, J307 to J305, Z3-301 to Z3-4, Z301 to Z30, Z308 to Z306
Connections:
- net GND: now also C8.1, R337.2
- net VCC: now also R309.1, R336.2
- net V_SYNC_PULSE(50Hz): now also Z309.3 (C); no longer J302.3 (Pin_3)
- net ~{IOREQ}: now also Z301.9
- net ~{M1}: now also Z301.10
- net ~{WAIT}: now also C8.2, R309.2, R338.1; no longer E301.26 (~{WAIT})
- net at Z301.8: now also Z309.4 (~{S})
- new net: R337.1, Z309.2 (D)
- new net: D303.2 (A), D304.2 (A), R338.2
- new net: R336.1, Z309.1 (~{R})
- new net: J302.3 (Pin_3), Z309.5 (Q)
- new net ~{WAIT_EXT}: D304.1 (K), E301.26 (~{WAIT})
- new net ~{WAIT_IN}: D303.1 (K)
- no-connect marks 13 -> 19
Other:
- moved on the sheet: C23, D12, J301, J302, R12, R301, RST301, Z301C, Z30B

Commit message: Change Address decode to speed up the use of /WAIT to avoid conflicts when setting up character RAM. Rerange priority on Internal external /WAIT. Reconnect Clock to rest of circuit.
Signed-off-by: John Bradley <flypie@rocketmail.com>
Parts:
- removed unit 6 of Z30
- removed unit 4 of Z301
- added Z22: SN74ACT11N, Package_DIP:DIP-14_W7.62mm, symbol 74xx-FIX:74LS11
- added Z310: SN74AHCT08PWR, Package_SO:TSSOP-14_4.4x5mm_P0.65mm, symbol 74xx-FIX:74LS08
- C8: value 47pf -> 100pf
- R309: value 2K -> 1K
- R338: value 330 -> 150
Connections:
- no-connect marks 19 -> 21
Other:
- moved on the sheet: C8, D303, D304, J302, Logo301, Logo302, R306, R307, R308, R309, R336, R337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
