File: KiCad/ACE5/ACE5.sch (KiCad schematic (older format))
At the start: 24 parts, among them X2 32MHz

Commit message: Update ACE3NOKB to reflect errors in Mem Decode. ACE5NOKB test SMT ideas. Added 180 & 380.
Signed-off-by: John Bradley <flypie@rocketmail.com>
Parts:
- removed Z19: 74AHCT00, Package_DIP:DIP-14_W7.62mm_Socket, symbol 74xx:74LS00
- removed Z23: 74AHCT86, Package_DIP:DIP-14_W7.62mm_Socket, symbol 74xx:74LS86
- C100, C101: footprint Capacitor_THT:C_Disc_D3.0mm_W1.6mm_P2.50mm -> Capacitor_SMD:C_1206_3216Metric
- C7: footprint Capacitor_THT:CP_Radial_D4.0mm_P1.50mm -> Capacitor_Tantalum_SMD:CP_EIA-3528-21_Kemet-B_Pad1.50x2.35mm_HandSolder
- R25: footprint Resistor_THT:R_Axial_DIN0204_L3.6mm_D1.6mm_P1.90mm_Vertical -> Resistor_SMD:R_1206_3216Metric
- R32: footprint Resistor_THT:R_Axial_DIN0204_L3.6mm_D1.6mm_P2.54mm_Vertical -> Resistor_SMD:R_1206_3216Metric
- X2: footprint Crystal:Crystal_HC49-U_Vertical -> Crystal:Crystal_SMD_7050-2Pin_7.0x5.0mm
- Z0: footprint Package_QFP:PQFP-100_14x20mm_P0.65mm -> Package_QFP:LQFP-100_14x14mm_P0.5mm; symbol Zilog_Z80:Z84C15-QFP -> Zilog_Z80:Z84C15-VQFP
- Z22, Z25, Z404: footprint Package_DIP:DIP-14_W7.62mm_Socket -> Package_SO:SOIC-14_3.9x8.7mm_P1.27mm
- Z306: footprint Package_DIP:DIP-14_W7.62mm_Socket -> Package_SO:SOIC-16_3.9x9.9mm_P1.27mm
- Z307: footprint Package_DIP:DIP-16_W7.62mm_Socket -> Package_SO:SOIC-16_3.9x9.9mm_P1.27mm
- Z80CPUOUT1: footprint Connector_PinHeader_2.54mm:PinHeader_2x22_P2.54mm_Vertical -> Connector_PinHeader_2.54mm:PinHeader_2x22_P2.54mm_Vertical_SMD
Connections:
- net A0: now also Z0.3 (A0); no longer Z0.6 (A0)
- net A1: now also Z0.2 (A1); no longer Z0.5 (A1)
- net A10: now also Z0.93 (A10); no longer Z0.96 (A10)
- net A11: now also Z0.92 (A11); no longer Z0.95 (A11)
- net A12: now also Z0.91 (A12); no longer Z0.94 (A12)
- net A13: now also Z0.90 (A13); no longer Z0.93 (A13)
- net A14: now also Z0.89 (A14); no longer Z0.92 (A14)
- net A15: now also Z0.88 (A15); no longer Z0.91 (A15)
- net A2: now also Z0.1 (A2); no longer Z0.4 (A2)
- net A3: now also Z0.100 (A3); no longer Z0.3 (A3)
- net A4: now also Z0.99 (A4); no longer Z0.2 (A4)
- net A5: now also Z0.98 (A5); no longer Z0.1 (A5)
- net A6: now also Z0.97 (A6); no longer Z0.100 (A6)
- net A7: now also Z0.96 (A7); no longer Z0.99 (A7)
- net A8: now also Z0.95 (A8); no longer Z0.98 (A8)
- net A9: now also Z0.94 (A9); no longer Z0.97 (A9)
- net DA0: now also Z0.86 (D0); no longer Z0.89 (D0)
- net DA1: now also Z0.85 (D1); no longer Z0.88 (D1)
- net DA2: now also Z0.84 (D2); no longer Z0.87 (D2)
- net DA3: now also Z0.83 (D3); no longer Z0.86 (D3)
- net DA4: now also Z0.82 (D4); no longer Z0.85 (D4)
- net DA5: now also Z0.81 (D5); no longer Z0.84 (D5)
- net DA6: now also Z0.80 (D6); no longer Z0.83 (D6)
- net DA7: now also Z0.79 (D7); no longer Z0.82 (D7)
- net GND: now also Z0.13 (Vss), Z0.61 (Vss); no longer Z0.16 (VSS$1), Z0.67 (EV)
- net PHI: now also Z0.65 (CLKOUT), Z0.66 (CLKIN); no longer Z0.68 (CLKOUT), Z0.69 (CLKIN)
- net VCC: now also Z0.38 (Vcc), Z0.69 (IE1), Z0.87 (Vcc); no longer Z0.41 (VCC$1), Z0.72 (IEI), Z0.90 (VCC$2)
- net ~BUSAK: now also Z0.9 (/BUSACK); no longer Z0.12 (/BUSACK)
- net ~BUSRQ: now also Z0.7 (/BUSREQ); no longer Z0.10 (/BUSREQ)
- net ~HALT: now also Z0.15 (/HALT); no longer Z0.18 (/HALT)
- net ~INT: now also Z0.16 (/INT); no longer Z0.19 (/INT)
- net ~IOREQ: now also Z0.12 (/IORQ); no longer Z0.15 (/IORQ)
- net ~M1: now also Z0.5 (/M1); no longer Z0.8 (/M1)
- net ~MREQ: now also Z0.14 (/MREQ); no longer Z0.17 (/MREQ)
- net ~NMI: now also Z0.60 (/NMI); no longer Z0.63 (/NMI)
- net ~RD: now also Z0.11 (/RD); no longer Z0.14 (/RD)
- net ~REFSH: now also Z0.4 (/RFSH); no longer Z0.7 (/RFSH)
- net ~RESET: now also Z0.6 (/RESET); no longer Z0.9 (/RESET)
- net ~WAIT: now also Z0.8 (/WAIT); no longer Z0.11 (/WAIT)
- net ~WR: now also Z0.10 (/WR); no longer Z0.13 (/WR)
- net at C100.2, X2.1: now also Z0.63 (XTAL2); no longer Z0.66 (XTAL2)
- net at C101.2, X2.2: now also Z0.62 (XTAL1); no longer Z0.65 (XTAL1)
- no-connect marks 35 -> 20
Changed lines of the file:
@@
 Text Label 11100 2700 0    50   ~ 0
 ~WE
-NoConn ~ -1300 650
-NoConn ~ -1300 850
-NoConn ~ -700 750
-NoConn ~ -1450 750
-NoConn ~ -2050 850
-NoConn ~ -2050 650
 NoConn ~ 10000 4350
 $Sheet
-S 475  9500 1025 1000
+S 1500 9500 1000 1000
 U 5DD74AB7
 F0 "KIO" 118
@@
 $EndSheet
 $Sheet
-S 2000 9500 1000 1000
+S 3500 9500 1000 1000
 U 5DAF6158
 F0 "VDG" 118
@@
 F 0 "R25" H 4210 1480 50  0000 L BNN
 F 1 "220k" H 4250 1195 50  0000 L BNN
-F 2 "Resistor_THT:R_Axial_DIN0204_L3.6mm_D1.6mm_P1.90mm_Vertical" H 4400 1350 50  0001 C CNN
+F 2 "Resistor_SMD:R_1206_3216Metric" H 4400 1350 50  0001 C CNN
 F 3 "" H 4400 1350 50  0001 C CNN
 	1    4400 1350
@@
 $EndComp
 $Comp
-L Zilog_Z80:Z84C15-QFP Z0
+L Zilog_Z80:Z84C15-VQFP Z0
 U 1 1 5F80C8F8
 P 2400 1000
 F 0 "Z0" H 2800 1200 50  0000 C CNN
 F 1 "Z84C15QFP100" H 2800 1100 50  0000 C CNN
-F 2 "Package_QFP:PQFP-100_14x20mm_P0.65mm" H 2400 1000 50  0001 C CNN
+F 2 "Package_QFP:LQFP-100_14x14mm_P0.5mm" H 2400 1000 50  0001 C CNN
 F 3 "" H 2400 1000 50  0001 C CNN
 	1    2400 1000
@@
 F 0 "Z80CPUOUT1" H 1350 3250 50  0000 C CNN
 F 1 "Conn_02x22_Odd_Even" H 1350 3150 50  0000 C CNN
-F 2 "Connector_PinHeader_2.54mm:PinHeader_2x22_P2.54mm_Vertical" H 1300 2000 50  0001 C CNN
+F 2 "Connector_PinHeader_2.54mm:PinHeader_2x22_P2.54mm_Vertical_SMD" H 1300 2000 50  0001 C CNN
 F 3 "~" H 1300 2000 50  0001 C CNN
 	1    1300 2000
-	1    0    0    -1
-$EndComp
-$Comp
-L 74xx:74LS86 Z23
-U 1 1 6061F7ED
-P -1750 750
-F 0 "Z23" H -1750 1100 50  0000 C CNN
-F 1 "74AHCT86" H -1750 1000 50  0000 C CNN
-F 2 "Package_DIP:DIP-14_W7.62mm_Socket" H -1750 750 50  0001 C CNN
-F 3 "74xx~74ls86.pdf" H -1750 750 50  0001 C CNN
-	1    -1750 750
-	1    0    0    -1
-$EndComp
-$Comp
-L 74xx:74LS86 Z23
-U 2 1 60628B03
-P -1000 750
-F 0 "Z23" H -1000 1100 50  0000 C CNN
-F 1 "74AHCT86" H -1000 1000 50  0000 C CNN
-F 2 "Package_DIP:DIP-14_W7.62mm_Socket" H -1000 750 50  0001 C CNN
-F 3 "74xx~74ls86.pdf" H -1000 750 50  0001 C CNN
-	2    -1000 750
 	1    0    0    -1
 $EndComp
@@
 F 0 "C7" H 4445 1869 50  0000 L BNN
 F 1 "1U" H 4245 1869 50  0000 L BNN
-F 2 "Capacitor_THT:CP_Radial_D4.0mm_P1.50mm" H 4400 1850 50  0001 C CNN
+F 2 "Capacitor_Tantalum_SMD:CP_EIA-3528-21_Kemet-B_Pad1.50x2.35mm_HandSolder" H 4400 1850 50  0001 C CNN
 F 3 "" H 4400 1850 50  0001 C CNN
 	1    4400 1850
@@
 F 0 "C101" V 4900 2300 50  0000 C CNN
 F 1 "33pf" V 4800 2300 50  0000 C CNN
-F 2 "Capacitor_THT:C_Disc_D3.0mm_W1.6mm_P2.50mm" H 4625 2300 50  0001 C CNN
+F 2 "Capacitor_SMD:C_1206_3216Metric" H 4625 2300 50  0001 C CNN
 F 3 "" H 4625 2300 50  0001 C CNN
 	1    4625 2300
@@
 F 0 "X2" V 4975 2275 50  0000 R CNN
 F 1 "32MHz" V 4875 2275 50  0000 R CNN
-F 2 "Crystal:Crystal_HC49-U_Vertical" H 4900 2450 50  0001 C CNN
+F 2 "Crystal:Crystal_SMD_7050-2Pin_7.0x5.0mm" H 4900 2450 50  0001 C CNN
 F 3 "" H 4900 2450 50  0001 C CNN
 	1    4900 2450
@@
 F 0 "C100" V 4450 2575 50  0000 C CNN
 F 1 "33pf" V 4350 2575 50  0000 C CNN
-F 2 "Capacitor_THT:C_Disc_D3.0mm_W1.6mm_P2.50mm" H 4625 2600 50  0001 C CNN
+F 2 "Capacitor_SMD:C_1206_3216Metric" H 4625 2600 50  0001 C CNN
 F 3 "" H 4625 2600 50  0001 C CNN
 	1    4625 2600
@@
 $EndComp
 $Comp
-L Zilog_Z80:Z84C15-QFP Z0
+L Zilog_Z80:Z84C15-VQFP Z0
 U 2 1 5F80CEF0
 P 5400 2000
 F 0 "Z0" H 5850 2250 50  0000 C CNN
 F 1 "Z84C15QFP100" H 5850 2100 50  0000 C CNN
-F 2 "Package_QFP:PQFP-100_14x20mm_P0.65mm" H 5400 2000 50  0001 C CNN
+F 2 "Package_QFP:LQFP-100_14x14mm_P0.5mm" H 5400 2000 50  0001 C CNN
 F 3 "" H 5400 2000 50  0001 C CNN
 	2    5400 2000
@@
 F 0 "Z306" H 7945 4690 50  0000 C CNN
 F 1 "74AHCT04" H 7945 4590 50  0000 C CNN
-F 2 "Package_DIP:DIP-14_W7.62mm_Socket" H 7900 4350 50  0001 C CNN
+F 2 "Package_SO:SOIC-16_3.9x9.9mm_P1.27mm" H 7900 4350 50  0001 C CNN
 F 3 "http:~/www.ti.com/lit/gpn/sn74LS04" H 7900 4350 50  0001 C CNN
 	2    7900 4350
@@
 F 0 "Z25" H -1705 3610 50  0000 C CNN
 F 1 "74AHCT02" H -1705 3510 50  0000 C CNN
-F 2 "Package_DIP:DIP-14_W7.62mm_Socket" H -1750 3250 50  0001 C CNN
+F 2 "Package_SO:SOIC-14_3.9x8.7mm_P1.27mm" H -1750 3250 50  0001 C CNN
 F 3 "http:~/www.ti.com/lit/gpn/sn74ls02" H -1750 3250 50  0001 C CNN
 	3    -1750 3250
@@
 ~IOREQ
 $Sheet
-S 3500 9500 1000 1000
+S 3500 8000 1000 1000
 U 5DBBBE50
 F0 "IO&Speaker" 118
@@
 	7750 3300 7750 3250
 $Sheet
-S 5000 9500 1000 1000
+S 5500 9500 1000 1000
 U 5DC61528
 F0 "MMU" 118
@@
 MA19
 $Sheet
-S 6500 9500 1000 1000
+S 7500 9500 1000 1000
 U 5DE39253
 F0 "PSU" 118
@@
 $EndSheet
 $Sheet
-S 8000 9500 1000 1000
+S 9500 9500 1000 1000
 U 601C6FA0
 F0 "ADDRDECODE" 118
@@
 F 0 "Z404" H -1750 2450 50  0000 C CNN
 F 1 "74LS21" H -1750 2350 50  0000 C CNN
-F 2 "Package_DIP:DIP-14_W7.62mm_Socket" H -1750 2050 50  0001 C CNN
+F 2 "Package_SO:SOIC-14_3.9x8.7mm_P1.27mm" H -1750 2050 50  0001 C CNN
 F 3 "http://www.ti.com/lit/gpn/sn74LS21" H -1750 2050 50  0001 C CNN
 	2    -1750 2050
@@
 F 0 "R32" V 10625 2725 50  0000 C CNN
 F 1 "1K0" V 10725 2725 50  0000 C CNN
-F 2 "Resistor_THT:R_Axial_DIN0204_L3.6mm_D1.6mm_P2.54mm_Vertical" V 10780 2700 50  0001 C CNN
+F 2 "Resistor_SMD:R_1206_3216Metric" V 10780 2700 50  0001 C CNN
 F 3 "~" H 10850 2700 50  0001 C CNN
 	1    10850 2700
@@
 NoConn ~ -2050 2100
 NoConn ~ -2050 2200
-NoConn ~ -600 650
-NoConn ~ -600 850
-NoConn ~ 0    750
-$Comp
-L 74xx:74LS86 Z23
-U 3 1 6100DA9E
-P -300 750
-F 0 "Z23" H -300 1100 50  0000 C CNN
-F 1 "74AHCT86" H -300 1000 50  0000 C CNN
-F 2 "Package_DIP:DIP-14_W7.62mm_Socket" H -300 750 50  0001 C CNN
-F 3 "74xx~74ls86.pdf" H -300 750 50  0001 C CNN
-	3    -300 750
-	1    0    0    -1
-$EndComp
-$Comp
-L 74xx:74LS11 Z?
+$Comp
+L 74xx:74LS11 Z22
 U 3 1 610C57CB
 P -1750 2650
-AR Path="/5DAF6158/610C57CB" Ref="Z?"  Part="2"
-AR Path="/610C57CB" Ref="Z22"  Part="3"
 F 0 "Z22" H -1750 3030 50  0000 C CNN
 F 1 "74AHCT11" H -1750 2930 50  0000 C CNN
-F 2 "Package_DIP:DIP-14_W7.62mm_Socket" H -1750 2650 50  0001 C CNN
+F 2 "Package_SO:SOIC-14_3.9x8.7mm_P1.27mm" H -1750 2650 50  0001 C CNN
 F 3 "http:~/www.ti.com/lit/gpn/sn74AHCT11" H -1750 2650 50  0001 C CNN
 	3    -1750 2650
@@
 NoConn ~ -2050 2650
 NoConn ~ -2050 2750
-$Comp
-L 74xx:74LS00 Z?
-U 3 1 61203101
-P -1700 1400
-AR Path="/601C6FA0/61203101" Ref="Z?"  Part="3"
-AR Path="/61203101" Ref="Z19"  Part="3"
-F 0 "Z19" H -1685 1750 50  0000 C CNN
-F 1 "74AHCT00" H -1685 1650 50  0000 C CNN
-F 2 "Package_DIP:DIP-14_W7.62mm_Socket" H -1700 1400 50  0001 C CNN
-F 3 "http://www.ti.com/lit/gpn/sn74ls00" H -1700 1400 50  0001 C CNN
-F 4 "SN74AHCT00N" H -1700 1400 50  0001 C CNN "Manufacturer_Part_Number"
-F 5 "Texas Instruments" H -1700 1400 50  0001 C CNN "Manufacturer_Name"
-	3    -1700 1400
-	1    0    0    -1
-$EndComp
-NoConn ~ -1400 1400
-NoConn ~ -2000 1500
-NoConn ~ -2000 1300
-$Comp
-L 74xx:74LS00 Z19
-U 4 1 61294137
-P -950 1400
-AR Path="/61294137" Ref="Z19"  Part="4"
-AR Path="/606B9078/61294137" Ref="Z?"  Part="4"
-AR Path="/601C6FA0/61294137" Ref="Z?"  Part="4"
-F 0 "Z19" H -925 1750 50  0000 C CNN
-F 1 "74AHCT00" H -925 1650 50  0000 C CNN
-F 2 "Package_DIP:DIP-14_W7.62mm_Socket" H -950 1400 50  0001 C CNN
-F 3 "http://www.ti.com/lit/gpn/sn74ls00" H -950 1400 50  0001 C CNN
-F 4 "SN74AHCT00N" H -950 1400 50  0001 C CNN "Manufacturer_Part_Number"
-F 5 "Texas Instruments" H -950 1400 50  0001 C CNN "Manufacturer_Name"
-	4    -950 1400
-	1    0    0    -1
-$EndComp
-NoConn ~ -650 1400
-NoConn ~ -1250 1500
-NoConn ~ -1250 1300
 Wire Wire Line
 	8400 5050 8400 4950
@@
 F 0 "Z307" H 9575 4875 50  0000 C CNN
 F 1 "74AHCT139" H 9575 4775 50  0000 C CNN
-F 2 "Package_DIP:DIP-16_W7.62mm_Socket" H 9500 4450 50  0001 C CNN
+F 2 "Package_SO:SOIC-16_3.9x9.9mm_P1.27mm" H 9500 4450 50  0001 C CNN
 F 3 "http://www.ti.com/lit/gpn/sn74LS139" H 9500 4450 50  0001 C CNN
 	2    9500 4450
@@
 $EndComp
 $Sheet
-S 9500 9500 1000 900
+S 1500 8000 1000 900
 U 604875AE
 F0 "STM8SUBSYS" 118
