File: KiCad/ACEZ180/KIO.kicad_sch (KiCad schematic)
At the start: 6 parts, among them J300 Conn_02x06_Odd_Even, J301 Conn_02x05_Odd_Even, J303 Conn_02x03_Odd_Even, J304 Conn_02x05_Odd_Even, J501 Conn_02x05_Odd_Even, J502 Conn_02x03_Odd_Even

Commit message: Fix mistake with ROM Select.
Signed-off-by: John Bradley <flypie@rocketmail.com>
Parts:
- J300: footprint (none) -> Connector_PinHeader_2.54mm:PinHeader_2x06_P2.54mm_Vertical
- J301, J304, J501: footprint (none) -> Connector_PinHeader_2.54mm:PinHeader_2x05_P2.54mm_Vertical
- J303, J502: footprint (none) -> Connector_PinHeader_2.54mm:PinHeader_2x03_P2.54mm_Vertical
Changed lines of the file:
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@@
     (property "Reference" "J300" (id 0) (at 180.34 45.72 0))
     (property "Value" "Conn_02x06_Odd_Even" (id 1) (at 180.34 48.26 0))
-    (property "Footprint" "" (id 2) (at 179.07 57.15 0)
+    (property "Footprint" "Connector_PinHeader_2.54mm:PinHeader_2x06_P2.54mm_Vertical" (id 2) (at 179.07 57.15 0)
       (effects (font (size 1.27 1.27)) hide)
     )
@@
     (property "Reference" "J301" (id 0) (at 180.34 71.12 0))
     (property "Value" "Conn_02x05_Odd_Even" (id 1) (at 180.34 73.66 0))
-    (property "Footprint" "" (id 2) (at 179.07 82.55 0)
+    (property "Footprint" "Connector_PinHeader_2.54mm:PinHeader_2x05_P2.54mm_Vertical" (id 2) (at 179.07 82.55 0)
       (effects (font (size 1.27 1.27)) hide)
     )
@@
     (property "Reference" "J502" (id 0) (at 231.14 99.06 0))
     (property "Value" "Conn_02x03_Odd_Even" (id 1) (at 231.14 101.6 0))
-    (property "Footprint" "" (id 2) (at 229.87 107.95 0)
+    (property "Footprint" "Connector_PinHeader_2.54mm:PinHeader_2x03_P2.54mm_Vertical" (id 2) (at 229.87 107.95 0)
       (effects (font (size 1.27 1.27)) hide)
     )
@@
     (property "Reference" "J501" (id 0) (at 180.34 95.25 0))
     (property "Value" "Conn_02x05_Odd_Even" (id 1) (at 180.34 97.79 0))
-    (property "Footprint" "" (id 2) (at 179.07 106.68 0)
+    (property "Footprint" "Connector_PinHeader_2.54mm:PinHeader_2x05_P2.54mm_Vertical" (id 2) (at 179.07 106.68 0)
       (effects (font (size 1.27 1.27)) hide)
     )
@@
     (property "Reference" "J303" (id 0) (at 231.14 45.72 0))
     (property "Value" "Conn_02x03_Odd_Even" (id 1) (at 231.14 48.26 0))
-    (property "Footprint" "" (id 2) (at 229.87 54.61 0)
+    (property "Footprint" "Connector_PinHeader_2.54mm:PinHeader_2x03_P2.54mm_Vertical" (id 2) (at 229.87 54.61 0)
       (effects (font (size 1.27 1.27)) hide)
     )
@@
     (property "Reference" "J304" (id 0) (at 231.14 71.12 0))
     (property "Value" "Conn_02x05_Odd_Even" (id 1) (at 231.14 73.66 0))
-    (property "Footprint" "" (id 2) (at 229.87 82.55 0)
-      (effects (font (size 1.27 1.27)) hide)
-    )
+    (property "Footprint" "Connector_PinHeader_2.54mm:PinHeader_2x05_P2.54mm_Vertical" (id 2) (at 229.87 82.55 0)
+      (effects (font (size 1.27 1.27)) hide)
+    )
