File: KiCad/ACEZ380/ADDRDECODE.sch (KiCad schematic (older format))
At the start: 13 parts

Commit message: Update ACE3NOKB to reflect errors in Mem Decode. ACE5NOKB test SMT ideas. Added 180 & 380.
Signed-off-by: John Bradley <flypie@rocketmail.com>
Parts:
- renumbered D602 to D?, D601 to D?, D603 to D?, D604 to D?, D605 to D?, D606 to D?, R621 to R?, Z404 to U?, Z407 to Z?, Z306 to Z?
Changed lines of the file:
@@
 U 1 1 6024C8EB
 P 7350 3150
-AR Path="/6024C8EB" Ref="Z?"  Part="1"
-AR Path="/601C6FA0/6024C8EB" Ref="Z407"  Part="1"
-AR Path="/601B22CC/6024C8EB" Ref="Z407"  Part="1"
 F 0 "Z407" H 7375 3575 50  0000 C CNN
 F 1 "74AHCT30D" H 7375 3475 50  0000 C CNN
@@
 U 1 1 605A9444
 P 9950 2450
-AR Path="/605A9444" Ref="U?"  Part="1"
-AR Path="/601C6FA0/605A9444" Ref="Z404"  Part="1"
-AR Path="/601B22CC/605A9444" Ref="Z404"  Part="1"
 F 0 "Z404" H 9950 2800 50  0000 C CNN
 F 1 "74LS21" H 9950 2750 50  0000 C CNN
@@
 U 1 1 605721B4
 P 3700 1650
-AR Path="/605721B4" Ref="#~~~PWR?"  Part="1"
-AR Path="/601B22CC/605721B4" Ref="#~~~PWR0101"  Part="1"
 F 0 "#~~~PWR0101" H 3700 1400 50  0001 C CNN
 F 1 "GND" V 3735 1515 50  0000 R CNN
@@
 U 1 1 605721BB
 P 3225 850
-AR Path="/5D66C06C/605721BB" Ref="D?"  Part="1"
-AR Path="/605721BB" Ref="D?"  Part="1"
-AR Path="/601B22CC/605721BB" Ref="D602"  Part="1"
 F 0 "D602" V 3145 800 50  0000 L CNN
 F 1 "1N4148" V 3225 935 50  0001 L CNN
@@
 U 1 1 605721C1
 P 3475 750
-AR Path="/5D66C06C/605721C1" Ref="D?"  Part="1"
-AR Path="/605721C1" Ref="D?"  Part="1"
-AR Path="/601B22CC/605721C1" Ref="D601"  Part="1"
 F 0 "D601" V 3395 700 50  0000 L CNN
 F 1 "1N4148" V 3475 835 50  0001 L CNN
@@
 U 1 1 605721C7
 P 3475 950
-AR Path="/5D66C06C/605721C7" Ref="D?"  Part="1"
-AR Path="/605721C7" Ref="D?"  Part="1"
-AR Path="/601B22CC/605721C7" Ref="D603"  Part="1"
 F 0 "D603" V 3395 900 50  0000 L CNN
 F 1 "1N4148" V 3475 1035 50  0001 L CNN
@@
 U 1 1 605721CD
 P 3225 1050
-AR Path="/5D66C06C/605721CD" Ref="D?"  Part="1"
-AR Path="/605721CD" Ref="D?"  Part="1"
-AR Path="/601B22CC/605721CD" Ref="D604"  Part="1"
 F 0 "D604" V 3145 1000 50  0000 L CNN
 F 1 "1N4148" V 3225 1135 50  0001 L CNN
@@
 U 1 1 605721D3
 P 3475 1150
-AR Path="/5D66C06C/605721D3" Ref="D?"  Part="1"
-AR Path="/605721D3" Ref="D?"  Part="1"
-AR Path="/601B22CC/605721D3" Ref="D605"  Part="1"
 F 0 "D605" V 3395 1100 50  0000 L CNN
 F 1 "1N4148" V 3475 1235 50  0001 L CNN
@@
 U 1 1 605721D9
 P 3225 1250
-AR Path="/5D66C06C/605721D9" Ref="D?"  Part="1"
-AR Path="/605721D9" Ref="D?"  Part="1"
-AR Path="/601B22CC/605721D9" Ref="D606"  Part="1"
 F 0 "D606" V 3145 1200 50  0000 L CNN
 F 1 "1N4148" V 3225 1335 50  0001 L CNN
@@
 U 1 1 605721DF
 P 3700 1400
-AR Path="/605721DF" Ref="R?"  Part="1"
-AR Path="/601B22CC/605721DF" Ref="R621"  Part="1"
 F 0 "R621" H 3775 1475 59  0000 L CNN
 F 1 "10" H 3775 1375 59  0000 L CNN
@@
 U 1 1 605721E5
 P 4200 1000
-AR Path="/605721E5" Ref="Z?"  Part="6"
-AR Path="/601B22CC/605721E5" Ref="Z306"  Part="1"
 F 0 "Z306" H 4245 1340 50  0000 C CNN
 F 1 "SN74AHCT04N" H 4245 1240 50  0000 C CNN
