File: KiCad/ACEZ380/acez380.sch (KiCad schematic (older format))
At the start: 21 parts, among them J607 Conn_02x04_Odd_Even, X2 20MHz

Commit message: Update ACE3NOKB to reflect errors in Mem Decode. ACE5NOKB test SMT ideas. Added 180 & 380.
Signed-off-by: John Bradley <flypie@rocketmail.com>
Parts:
- renumbered J607 to J?, Z306 to Z?
Changed lines of the file:
@@
 U 2 1 61E77BBF
 P 7900 4650
-AR Path="/5D66C06C/61E77BBF" Ref="Z?"  Part="5"
-AR Path="/61E77BBF" Ref="Z306"  Part="2"
 F 0 "Z306" H 7925 5025 50  0000 C CNN
 F 1 "SN74AHCT04N" H 7925 4925 50  0000 C CNN
@@
 U 2 1 6068E00B
 P -1300 2350
-AR Path="/6068E00B" Ref="Z600"  Part="2"
-AR Path="/5EDE0D3D/6068E00B" Ref="Z?"  Part="1"
 F 0 "Z600" H -1300 2775 50  0000 C CNN
 F 1 "SN74AHCT139N" H -1300 2675 50  0000 C CNN
@@
 U 1 1 60B41C8E
 P 5900 2900
-AR Path="/601B2B8F/60B41C8E" Ref="J?"  Part="1"
-AR Path="/60B41C8E" Ref="J607"  Part="1"
 F 0 "J607" H 5975 3250 50  0000 C CNN
 F 1 "Conn_02x04_Odd_Even" H 5975 3150 50  0000 C CNN
@@
 U 1 1 60B41C95
 P 6300 3100
-AR Path="/601B2B8F/60B41C95" Ref="#PWR?"  Part="1"
-AR Path="/60B41C95" Ref="#PWR0121"  Part="1"
 F 0 "#PWR0121" H 6300 2850 50  0001 C CNN
 F 1 "GND" V 6350 2950 50  0000 R CNN
@@
 U 1 1 60B41C9C
 P 5600 3100
-AR Path="/601B2B8F/60B41C9C" Ref="#PWR?"  Part="1"
-AR Path="/60B41C9C" Ref="#PWR0122"  Part="1"
 F 0 "#PWR0122" H 5600 2950 50  0001 C CNN
 F 1 "VCC" V 5450 3100 50  0000 C CNN
