File: KiCad/PS2TestCard/PS2TestCard.kicad_pcb (KiCad board)
At the start: 2 copper layers, 75.6 x 69.2 mm, 13 parts, among them J2 Conn_02x06_Counter_Clockwise, P1 Mini-DIN-6, P2 Mini-DIN-6

Commit message: First complete system. Unlikely to work but will serve as the basis of a system to test VGA.
Signed-off-by: John Bradley <flypie@rocketmail.com>
Connections:
- net /~BUSAK renamed /~{BUSAK}
- net /~BUSRQ renamed /~{BUSRQ}
- net /~CPUCLK renamed /~{CPUCLK}
- net /~HALT renamed /~{HALT}
- net /~INT renamed /~{INT}
- net /~IOREQ renamed /~{IOREQ}
- net /~M1 renamed /~{M1}
- net /~MREQ renamed /~{MREQ}
- net /~NMI renamed /~{NMI}
- net /~Q renamed /~{Q}
- net /~RD renamed /~{RD}
- net /~REFSH renamed /~{REFSH}
- net /~RESET renamed /~{RESET}
- net /~WAIT renamed /~{WAIT}
- net /~WE renamed /~{WE}
- net /~WR renamed /~{WR}
- J2 pad 10: Net-(J2-Pad10) -> unconnected-(J2-Pad10)
- J2 pad 11: Net-(J2-Pad11) -> unconnected-(J2-Pad11)
- J2 pad 12: Net-(J2-Pad12) -> unconnected-(J2-Pad12)
- J2 pad 6: Net-(J2-Pad6) -> unconnected-(J2-Pad6)
- J2 pad 7: Net-(J2-Pad7) -> unconnected-(J2-Pad7)
- J2 pad 8: Net-(J2-Pad8) -> unconnected-(J2-Pad8)
- J2 pad 9: Net-(J2-Pad9) -> unconnected-(J2-Pad9)
- P1 pad 2: Net-(P1-Pad2) -> unconnected-(P1-Pad2)
- P1 pad 6: Net-(P1-Pad6) -> unconnected-(P1-Pad6)
- P2 pad 2: Net-(P2-Pad2) -> unconnected-(P2-Pad2)
- P2 pad 6: Net-(P2-Pad6) -> unconnected-(P2-Pad6)
- Z1 pad 11: Net-(Z1-Pad11) -> unconnected-(Z1-Pad11)
- Z1 pad 12: Net-(Z1-Pad12) -> unconnected-(Z1-Pad12)
- Z1 pad 13: Net-(Z1-Pad13) -> unconnected-(Z1-Pad13)
- Z110 pad 10: Net-(Z110-Pad10) -> (no net)
- Z110 pad 13: Net-(Z110-Pad13) -> (no net)
- Z110 pad 9: Net-(Z110-Pad9) -> (no net)
- Z1101 pad 9: Net-(Z1101-Pad9) -> unconnected-(Z1101-Pad9)
- Z111 pad 10: Net-(Z111-Pad10) -> unconnected-(Z111-Pad10)
- Z111 pad 11: Net-(Z111-Pad11) -> unconnected-(Z111-Pad11)
- Z111 pad 12: Net-(Z111-Pad12) -> unconnected-(Z111-Pad12)
- Z111 pad 13: Net-(Z111-Pad13) -> unconnected-(Z111-Pad13)
- Z111 pad 14: Net-(Z111-Pad14) -> unconnected-(Z111-Pad14)
- Z111 pad 15: Net-(Z111-Pad15) -> unconnected-(Z111-Pad15)
- Z111 pad 4: Net-(Z111-Pad4) -> unconnected-(Z111-Pad4)
- Z111 pad 5: Net-(Z111-Pad5) -> unconnected-(Z111-Pad5)
- Z111 pad 6: Net-(Z111-Pad6) -> unconnected-(Z111-Pad6)
- Z111 pad 9: Net-(Z111-Pad9) -> unconnected-(Z111-Pad9)
- Z80CPUIN1 pad 45: Net-(Z80CPUIN1-Pad45) -> unconnected-(Z80CPUIN1-Pad45)
- Z80CPUIN1 pad 46: Net-(Z80CPUIN1-Pad46) -> unconnected-(Z80CPUIN1-Pad46)
- Z80CPUIN1 pad 47: Net-(Z80CPUIN1-Pad47) -> unconnected-(Z80CPUIN1-Pad47)
- Z80CPUIN1 pad 48: Net-(Z80CPUIN1-Pad48) -> unconnected-(Z80CPUIN1-Pad48)
Other:
- net class Default removed
- net class PWR removed
