File: KiCad/eMultiUniBoard/eMultiUniBoard.kicad_pcb (KiCad board)
At the start: 2 copper layers, 75.6 x 68.6 mm, 5 parts

Commit message: First complete system. Unlikely to work but will serve as the basis of a system to test VGA.
Signed-off-by: John Bradley <flypie@rocketmail.com>
Connections:
- net /~BUSAK renamed /~{BUSAK}
- net /~BUSRQ renamed /~{BUSRQ}
- net /~CPUCLK renamed /~{CPUCLK}
- net /~HALT renamed /~{HALT}
- net /~INT renamed /~{INT}
- net /~IOREQ renamed /~{IOREQ}
- net /~M1 renamed /~{M1}
- net /~MREQ renamed /~{MREQ}
- net /~NMI renamed /~{NMI}
- net /~RD renamed /~{RD}
- net /~REFSH renamed /~{REFSH}
- net /~RESET renamed /~{RESET}
- net /~WAIT renamed /~{WAIT}
- net /~WE renamed /~{WE}
- net /~WR renamed /~{WR}
Other:
- net class Default removed
