File: KiCad/ACE4NOKB/ACE4NOKB.kicad_sch (KiCad schematic)
At the start: 32 parts, among them Q400 2N3904, Q401 2N2369, X400 CRYSTALHC49U-V 6.5MHz

Commit message: Fix mistake with ROM Select.
Signed-off-by: John Bradley <flypie@rocketmail.com>
Parts:
- removed C400: 30p, Capacitor_THT:C_Disc_D3.8mm_W2.6mm_P2.50mm, symbol Device:C_Small
- removed C401: 100p, Capacitor_THT:C_Disc_D5.0mm_W2.5mm_P5.00mm, symbol Device:C_Small
- removed C402: 47pF, Capacitor_THT:C_Disc_D3.0mm_W1.6mm_P2.50mm, symbol Device:C
- removed C7: 1uf, Capacitor_THT:CP_Radial_D5.0mm_P2.00mm, symbol Device:C_Polarized
- removed HBL1, HBR1, HTL1, HTR1: MountingHole, MountingHole:MountingHole_2.5mm, symbol Mechanical:MountingHole
- removed JZ80CPUOUT1: Conn_02x22_Odd_Even, Connector_PinHeader_2.54mm:PinHeader_2x22_P2.54mm_Vertical, symbol Connector_Generic:Conn_02x22_Odd_Even
- removed Q400: 2N3904, Package_TO_SOT_THT:TO-92_Inline, symbol Transistor_BJT:2N3904
- removed Q401: 2N2369, Package_TO_SOT_THT:TO-18-3, symbol Device:Q_NPN_EBC
- removed R25: 220k, Resistor_THT:R_Axial_DIN0204_L3.6mm_D1.6mm_P1.90mm_Vertical, symbol Device:R
- removed R3, R428: 400k, Resistor_THT:R_Axial_DIN0204_L3.6mm_D1.6mm_P1.90mm_Vertical, symbol Device:R
- removed R400: 4k7, Resistor_THT:R_Axial_DIN0204_L3.6mm_D1.6mm_P1.90mm_Vertical, symbol Device:R
- removed R401: 47k, Resistor_THT:R_Axial_DIN0204_L3.6mm_D1.6mm_P1.90mm_Vertical, symbol Device:R
- removed R402: 270R, Resistor_THT:R_Axial_DIN0204_L3.6mm_D1.6mm_P1.90mm_Vertical, symbol Device:R
- removed R403: 1K, Resistor_THT:R_Axial_DIN0204_L3.6mm_D1.6mm_P1.90mm_Vertical, symbol Device:R
- removed X400: CRYSTALHC49U-V 6.5MHz, Crystal:Crystal_HC49-U_Vertical, symbol Device:Crystal
- removed unit 3 of Z19
- removed Z22: 74HCT11, Package_DIP:DIP-14_W7.62mm_Socket, symbol 74xx:74LS11
- removed Z3-4: AS7C512 DIP/SOJ, Package_DIP:DIP-32_W7.62mm, symbol ExtraSymbols:AS7C512 DIP/SOJ
- removed Z306: 74AHCT04, Package_DIP:DIP-14_W7.62mm_Socket, symbol 74xx:74LS04
- removed Z307: 74AHCT139, Package_DIP:DIP-16_W7.62mm_Socket, symbol 74xx:74LS139
- removed Z308: 74HCT30, Package_DIP:DIP-14_W7.62mm_Socket, symbol 74xx:74LS30
- removed Z404: 74HCT21, Package_DIP:DIP-14_W7.62mm_Socket, symbol 74xx:74LS21
- added C22: 1 uf, Capacitor_THT:C_Disc_D3.0mm_W1.6mm_P2.50mm, symbol Device:C
- added C8: 2200pF, Capacitor_THT:C_Disc_D5.0mm_W2.5mm_P2.50mm, symbol Device:C
- added D300: 1N4148, Diode_THT:D_DO-35_SOD27_P2.54mm_Vertical_AnodeUp, symbol Diode:1N4148
- added E1: Conn_02x22_Odd_Even, Connector_PinHeader_2.54mm:PinHeader_2x22_P2.54mm_Vertical, symbol edg-con-ja:EDG-CON-JA-PIN
- added H1, H2, H3, H4: MountingHole, ExtraFootprints:MountingHole_3.5mm_with_Stencil_hole, symbol Mechanical:MountingHole
- added J310, J312, J313, J314, J405, J406: Conn_01x03, Connector_PinHeader_2.54mm:PinHeader_1x03_P2.54mm_Vertical, symbol Connector_Generic:Conn_01x03
- added J311: Conn_02x01_Odd_Even, Connector_PinHeader_2.54mm:PinHeader_2x01_P2.54mm_Vertical, symbol Connector_Generic:Conn_01x02
- added R12: 1k, Resistor_THT:R_Axial_DIN0204_L3.6mm_D1.6mm_P1.90mm_Vertical, symbol Device:R
- added R130, R131: 10K, Resistor_THT:R_Axial_DIN0204_L3.6mm_D1.6mm_P1.90mm_Vertical, symbol Device:R
- added R141: 10k, Resistor_THT:R_Axial_DIN0204_L3.6mm_D1.6mm_P1.90mm_Vertical, symbol Device:R
- added R301, R404: 500, Resistor_THT:R_Axial_DIN0204_L3.6mm_D1.6mm_P1.90mm_Vertical, symbol Device:R
- added R302: 100, Resistor_THT:R_Axial_DIN0204_L3.6mm_D1.6mm_P1.90mm_Vertical, symbol Device:R
- added R303, R406: 15K, Resistor_THT:R_Axial_DIN0204_L3.6mm_D1.6mm_P1.90mm_Vertical, symbol Device:R
- added RST1: TS02-66-60-BK-100-SCR-D, ExtraFootprints:TE Connectivity 1-1825910-4 Black Button Tactile Switch, Single Pole Single Throw (SPST), symbol ExtraSymbols:TE Connectivity 1-1825910-4 Black Button Tactile Switch, Single Po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
- added SW401: SW_SPDT, ExtraFootprints:B13AP, symbol Switch:SW_SPDT
- added X402: 6.5536 MHz, Crystal:Crystal_HC49-U_Vertical, symbol Device:Crystal
- added Z23: SN74AHCT86N, Package_DIP:DIP-14_W7.62mm, symbol 74xx:74LS86
- added Z25: SN74AHCT02, Package_DIP:DIP-14_W7.62mm, symbol 74xx:74LS02
- added Z3-4, Z309: IS62C256AL-45ULI, ExtraFootprints:SOP-28_8.3x18.15mm_P1.27mm, symbol ExtraSymbols:IS62C256AL
- added Z301: SN74AS21N, Package_DIP:DIP-14_W7.62mm, symbol 74xx-FIX:74LS21
- added Z306: SN74AHCT04N, Package_DIP:DIP-14_W7.62mm, symbol 74xx:74LS04
- added Z310: SN74AHCT32N, Package_DIP:DIP-14_W7.62mm, symbol 74xx:74LS32
- added Z402: 512MLF, Package_SO:SOIC-8_3.9x4.9mm_P1.27mm, symbol ExtraSymbols:512MLF
- Logo1, Logo2: Manufacturer_Name (none) -> logo; Manufacturer_Part_Number (none) -> logo
- R110: value 270 -> 10K; Manufacturer_Name Vishay -> (none); Manufacturer_Part_Number CCF07270RGKE36 -> (none)
- R24: value 10k -> 10K; Manufacturer_Name Vishay -> (none); Manufacturer_Part_Number MBA02040C1002FRP00 -> (none)
- Z0: value Z84C1516FSG -> Z80C15CPU_QFP
- Z1-2: value SST39SF010 -> SST39SF010A-45-4I-NHE; Manufacturer_Name Microchip Technology -> microchip; Manufacturer_Part_Number SST39SF010A-45-4I-NHE -> SST39SF010A-45-4I-NHE
- Z19: value 74AHCT00 -> SN74AHCT00N; footprint Package_DIP:DIP-14_W7.62mm_Socket -> Package_DIP:DIP-14_W7.62mm; Manufacturer_Name Texas Instruments -> (none); Manufacturer_Part_Number SN74AHCT00NE4 -> (none)
Connections:
- net +9Vsm: now also E1.39 (+9V)
- net A0: now also E1.7 (A0), Z3-4.10 (A0), Z309.10 (A0)
- net A1: now also E1.8 (A1), Z3-4.9 (A1), Z309.9 (A1)
- net A10: now also E1.15 (A10), Z3-4.21 (A10), Z309.21 (A10)
- net A11: now also E1.33 (A11), Z3-4.23 (A11), Z309.23 (A11)
- net A12: now also E1.31 (A12), Z3-4.2 (A12), Z309.2 (A12)
- net A13: now also E1.29 (A13), Z3-4.26 (A13), Z309.26 (A13)
- net A14: now also E1.27 (A14), Z3-4.1 (A14), Z309.1 (A14); no longer Z1-2.29 (A14)
- net A15: now also E1.25 (A15)
- net A2: now also E1.17 (A2), Z3-4.8 (A2), Z309.8 (A2)
- net A3: now also E1.10 (A3), Z3-4.7 (A3), Z309.7 (A3)
- net A4: now also E1.12 (A4), Z3-4.6 (A4), Z309.6 (A4)
- net A5: now also E1.14 (A5), Z3-4.5 (A5), Z309.5 (A5)
- net A6: now also E1.16 (A6), Z3-4.4 (A6), Z309.4 (A6)
- net A7: now also E1.9 (A7), Z3-4.3 (A7), Z309.3 (A7)
- net A8: now also E1.11 (A8), Z3-4.25 (A8), Z309.25 (A8)
- net A9: now also E1.13 (A9), Z3-4.24 (A9), Z309.24 (A9)
- net GND: now also Z0.65 (XTAL1), C22.2, C8.1, E1.41 (GND0), E1.43 (GND1), E1.44 (GND2), J311.2 (Pin_2), R301.1, R404.1, RST1.1, RST1.2, Z3-4.14 (GND), Z309.14 (GND), Z402.3 (GND)
- net PHI: now also E1.35 (~{CLK}), SW401.2 (B)
- net VCC: now also R24.2, D300.1 (K), E1.37 (+5V), R12.1, R130.1, R131.1, R141.1, R303.1, R406.1, Z3-4.28 (VCC), Z309.28 (VCC), Z402.2 (VDD); no longer R24.1
- net ~{BUSAK}: now also E1.28 (~{BUSACK})
- net ~{BUSRQ}: now also R24.1, E1.24 (~{BUSREQ}); no longer R24.2
- net ~{HALT}: now also E1.38 (~{HALT})
- net ~{INT}: now also Z0.19 (/INT), E1.42 (~{INT}), J310.2 (Pin_2), R130.2; no longer Z0.63 (/NMI)
- net ~{IOREQ}: now also E1.34 (~{IOREQ})
- net ~{M1}: now also E1.20 (~{M1})
- net ~{MREQ}: now also E1.36 (~{MREQ})
- net ~{NMI}: now also Z0.63 (/NMI), E1.40 (~{NMI}); no longer Z0.19 (/INT)
- net ~{RD}: now also E1.32 (~{RD}), Z3-4.22 (~{OE}), Z309.22 (~{OE}); no longer Z1-2.24 (OE)
- net ~{REFSH}: now also E1.18 (~{RFSH})
- net ~{RESET}: now also C22.1, D300.2 (A), E1.22 (~{RESET}), R12.2, R302.1
- net ~{WAIT}: now also C8.2, E1.26 (~{WAIT}), R131.2
- net ~{WE}: now also E1.1 (~{WE})
- net ~{WR}: now also E1.30 (~{WR}), Z3-4.27 (~{WE}), Z309.27 (~{WE})
- net UPPERROMSELECT1: now reaches Z1-2.3 (A15)
- net UPPERROMSELECT1: now also J313.2 (Pin_2); no longer Z1-2.2 (A16)
- net at Z1-2.31 (PGM): now also R141.2
- net DA0 renamed D0
- net D0: now also E1.6 (D0), Z3-4.11 (I/O0), Z309.11 (I/O0)
- net DA1 renamed D1
- net D1: now also E1.5 (D1), Z3-4.12 (I/O1), Z309.12 (I/O1)
- net DA2 renamed D2
- net D2: now also E1.4 (D2), Z3-4.13 (I/O2), Z309.13 (I/O2)
- net DA3 renamed D3
- net D3: now also E1.21 (D3), Z3-4.15 (I/O3), Z309.15 (I/O3)
- net DA4 renamed D4
- net D4: now also E1.23 (D4), Z3-4.16 (I/O4), Z309.16 (I/O4)
- net DA5 renamed D5
- net D5: now also E1.19 (D5), Z3-4.17 (I/O5), Z309.17 (I/O5)
- net DA6 renamed D6
- net D6: now also E1.3 (D6), Z3-4.18 (I/O6), Z309.18 (I/O6)
- net DA7 renamed D7
- net D7: now also E1.2 (D7), Z3-4.19 (I/O7), Z309.19 (I/O7)
- net ROM_SELECT: no longer names the net of Z1-2.22 (CE)
- net ROM_SELECT: now also Z1-2.24 (OE), Z301.8
- new net: J312.1 (Pin_1), J313.1 (Pin_1), J314.1 (Pin_1), R301.2
- new net: J312.3 (Pin_3), J313.3 (Pin_3), J314.3 (Pin_3), R303.2
- new net: J405.1 (Pin_1), J406.1 (Pin_1), R404.2
- new net: J405.3 (Pin_3), J406.3 (Pin_3), R406.2
- new net: J311.1 (Pin_1), R302.2, RST1.3, RST1.4
- new net: X402.2, Z402.1 (X1/CLK)
- new net: X402.1, Z402.8 (X2)
- new net FONTCHARX0: SW401.1 (A)
- new net S0: J405.2 (Pin_2), Z402.6 (S0)
- new net S1: J406.2 (Pin_2), Z402.7 (S1)
- new net TURBOCPUCLK: SW401.3 (C), Z402.5 (CLKOUT)
- new net UPPERROMSELECT0: J312.2 (Pin_2), Z1-2.29 (A14)
- new net UPPERROMSELECT2: J314.2 (Pin_2), Z1-2.2 (A16)
- new net VDGCLK: Z402.4 (REF)
- new net V_SYNC_PULSE(50Hz): J310.3 (Pin_3)
- new net ~{0000-1FFF}: Z301.13
- new net ~{3000-37FF}: Z301.10
- new net ~{3800-3BFF}: Z301.9
- new net ~{BOTTOM32KCS}: Z3-4.20 (~{CE})
- new net ~{CPU2FONTROMCS}: Z301.12
- new net ~{INTFROMKIO}: J310.1 (Pin_1)
- new net ~{TOP32KCS}: Z309.20 (~{CE})
- no-connect marks 31 -> 30
Other:
- added sheet Cascade (Cascade4040.kicad_sch)
- note added: "Added Pull up"
- note added: "Mode 2 via KIO"
- note added: "Orginal int. Straight to CPU."
- note added: "PIN Compatible with NB3N502DR2G Different Multiply Table"
- note added: "S0 S1 CLK 0 0 4X input M 0 5.333X input 1 0 5X input 0 M 2.5X input M M 2X input 1 M 3.333X input 0 1 6X input M 1 3X input 1 1 8X input 0 = connect directly to ground 1 = connect directly to VDD M = leave unconnected (floating)"
- note added: "VDGCLK_DIV_2"
- note removed: "~{IOREQ&11111111B}"
- title: ACE4NOKB -> JupiterAce Z80 plus KIO and new memory format.
- moved on the sheet: Z1-2

Commit message: Update to last expermintal version. Uses clock sythsiser and can be switched between full ACE compatible and inhanced IO. Should be able to switch between multiple ROM images tosred on the same chip.
Signed-off-by: John Bradley <flypie@rocketmail.com>
Parts:
- removed J405, J406: Conn_01x03, Connector_PinHeader_2.54mm:PinHeader_1x03_P2.54mm_Vertical, symbol Connector_Generic:Conn_01x03
- removed R404: 500, Resistor_THT:R_Axial_DIN0204_L3.6mm_D1.6mm_P1.90mm_Vertical, symbol Device:R
- removed R406: 15K, Resistor_THT:R_Axial_DIN0204_L3.6mm_D1.6mm_P1.90mm_Vertical, symbol Device:R
- removed RST1: TS02-66-60-BK-100-SCR-D, ExtraFootprints:TE Connectivity 1-1825910-4 Black Button Tactile Switch, Single Pole Single Throw (SPST), symbol ExtraSymbols:TE Connectivity 1-1825910-4 Black Button Tactile Switch, Single Po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
- removed SW401: SW_SPDT, ExtraFootprints:B13AP, symbol Switch:SW_SPDT
- removed X402: 6.5536 MHz, Crystal:Crystal_HC49-U_Vertical, symbol Device:Crystal
- removed Z25: SN74AHCT02, Package_DIP:DIP-14_W7.62mm, symbol 74xx:74LS02
- removed Z306: SN74AHCT04N, Package_DIP:DIP-14_W7.62mm, symbol 74xx:74LS04
- removed Z402: 512MLF, Package_SO:SOIC-8_3.9x4.9mm_P1.27mm, symbol ExtraSymbols:512MLF
- added J308, J309: Conn_01x03, Connector_PinHeader_2.54mm:PinHeader_1x03_P2.54mm_Vertical, symbol Connector_Generic:Conn_01x03
- added R1, R2: 4K7, Resistor_THT:R_Axial_DIN0204_L3.6mm_D1.6mm_P1.90mm_Vertical, symbol Device:R
- added R306, R307: R, Resistor_THT:R_Axial_DIN0204_L3.6mm_D1.6mm_P1.90mm_Vertical, symbol Device:R
- added RST1: TS02-66-60-BK-100-SCR-D, TS026660BK100SCRD, symbol ExtraSymbols:TS02-66-60-BK-100-SCR-D
- added SW302: EG2305, ExtraFootprints:SP112DP3T, symbol ExtraSymbols:SP112-DP3T
- added X1: 6.5536 MHz, Crystal:Crystal_HC49-U_Vertical, symbol Device:Crystal
- added Z306 (x2): SN74AHCT04N, Package_DIP:DIP-14_W7.62mm, symbol 74xx:74LS04
- added unit 3 of Z310
- added Z312: 512MLF, Package_SO:SOIC-8_3.9x4.9mm_P1.27mm, symbol ExtraSymbols:512MLF
- H1, H2, H3, H4: Manufacturer_Name hole -> (none); Manufacturer_Part_Number hole -> (none)
- Logo1, Logo2: Manufacturer_Name logo -> (none); Manufacturer_Part_Number logo -> (none)
- R131, R141: Manufacturer_Name Vishay -> (none); Manufacturer_Part_Number MBA02040C1002FRP00 -> (none)
- Z0: value Z80C15CPU_QFP -> Z84C15F-20x30; symbol Zilog_Z80:Z84C15-QFP_ALT1 -> CPU_Zilog_Z80:Z84C15F-20x30; Manufacturer_Name Zilog -> (none); Manufacturer_Part_Number Z84C00 -> (none)
- Z1-2: Manufacturer_Name microchip -> (none); Manufacturer_Part_Number SST39SF010A-45-4I-NHE -> (none)
- Z23: Manufacturer_Name Texas Instruments -> (none); Manufacturer_Part_Number SN74AHCT86N -> (none)
- Z3-4, Z309: Arrow Part Number (none) -> IS62C256AL-45ULI; Arrow Price/Stock (none) -> https://www.arrow.com/en/products/is62c256al-45uli/integrat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; Manufacturer_Name (none) -> Integrated Silicon Solution Inc.; Manufacturer_Part_Number (none) -> IS62C256AL-45ULI; Mouser Price/Stock (none) -> https://www.mouser.co.uk/ProductDetail/ISSI/IS62C256AL-45UL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
- Z301: Manufacturer_Name Texas Instruments -> (none); Manufacturer_Part_Number SN74AS21N -> (none)
Connections:
- net FONTCHARX0: now also SW302.4 (C), SW302.5 (C)
- net GND: now also R306.1, RST1.1 (NO_1), RST1.2 (NO_2), SW302.11 (M), SW302.12 (M), Z312.3 (GND); no longer Z0.16 (VSS$1), Z0.64 (VSS$2)
- net PHI: now also SW302.2 (COM), SW302.7 (COM)
- net S0: now also J308.2 (Pin_2), Z312.6 (S0)
- net S1: now also J309.2 (Pin_2), Z312.7 (S1)
- net TURBOCPUCLK: now also SW302.1 (A), SW302.8 (A), Z312.5 (CLKOUT)
- net VCC: now also R307.1, Z312.2 (VDD); no longer Z0.41 (VCC$1), Z0.90 (VCC$2)
- net at J311.1 (Pin_1), R302.2: now also RST1.3 (COM_1), RST1.4 (COM_2)
- new net: R1.1, R2.2, Z306.1, Z306.2
- new net: R2.1, X1.1, Z306.1
- new net: J308.1 (Pin_1), J309.1 (Pin_1), R306.2
- new net: J308.3 (Pin_3), J309.3 (Pin_3), R307.2
- new net: SW302.10 (M), SW302.9 (M)
- new net SHIFTCLK: R1.2, SW302.3 (B), SW302.6 (B), X1.2, Z306.2, Z312.1 (X1/CLK)
- no-connect marks 30 -> 34
Other:
- note removed: "VDGCLK_DIV_2"
- moved on the sheet: C22, C8, J310, J311, R131, R141, Z1-2, Z3-4, Z309

Commit message: Version with KIO replaced with Z84C15 and Video and Character RAM as MultiPorted.
Signed-off-by: John Bradley <flypie@rocketmail.com>
Parts:
- removed J308, J309: Conn_01x03, Connector_PinHeader_2.54mm:PinHeader_1x03_P2.54mm_Vertical, symbol Connector_Generic:Conn_01x03
- removed R1, R2: 4K7, Resistor_THT:R_Axial_DIN0204_L3.6mm_D1.6mm_P1.90mm_Vertical, symbol Device:R
- removed R306, R307: R, Resistor_THT:R_Axial_DIN0204_L3.6mm_D1.6mm_P1.90mm_Vertical, symbol Device:R
- removed SW302: EG2305, ExtraFootprints:SP112DP3T, symbol ExtraSymbols:SP112-DP3T
- removed X1: 6.5536 MHz, Crystal:Crystal_HC49-U_Vertical, symbol Device:Crystal
- removed Z23: SN74AHCT86N, Package_DIP:DIP-14_W7.62mm, symbol 74xx:74LS86
- removed Z306 (x2): SN74AHCT04N, Package_DIP:DIP-14_W7.62mm, symbol 74xx:74LS04
- removed Z310: SN74AHCT32N, Package_DIP:DIP-14_W7.62mm, symbol 74xx:74LS32
- removed Z312: 512MLF, Package_SO:SOIC-8_3.9x4.9mm_P1.27mm, symbol ExtraSymbols:512MLF
- added unit 3 of Z19
- added Z25: SN74AHCT02, Package_DIP:DIP-14_W7.62mm, symbol 74xx:74LS02
- H1, H2, H3, H4: now left out of the parts list
- RST1: footprint TS026660BK100SCRD -> ExtraFootprints:TS026660BK100SCRD
Connections:
- net VCC: now also R24.1; no longer R24.2
- net ~{BUSRQ}: now also R24.2; no longer R24.1
- net RESET_SW: now reaches J311.1 (Pin_1), R302.2, RST1.3 (COM_1), RST1.4 (COM_2)
- no-connect marks 34 -> 20
Other:
- added sheet CLOCK (Clock.kicad_sch)
- added sheet KEYBOARD (KEYBOARD.kicad_sch)
- note removed: "PIN Compatible with NB3N502DR2G Different Multiply Table"
- note removed: "S0 S1 CLK 0 0 4X input M 0 5.333X input 1 0 5X input 0 M 2.5X input M M 2X input 1 M 3.333X input 0 1 6X input M 1 3X input 1 1 8X input 0 = connect directly to ground 1 = connect directly to VDD M = leave unconnected (floating)"
- moved on the sheet: C22, C8, D300, J310, J311, J312, J313, J314, R110, R12, R130, R131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
